File: 65plus/65_plus/65_plus.kicad_pcb (KiCad board)
At the start: 2 copper layers, 352.4 x 104.8 mm, 91 parts, among them J1 USB_Type_C_2.0_Receptacle, P1 TC2030-IDC, SW0 K0, SW1 K0, SW10 K0, SW11 K0, SW12 K0, SW13 K0, SW14 K0, SW15 K0, SW16 K0, SW17 K0, SW18 K0, SW19 K0, SW2 K0, SW20 K0, SW21 K0, SW22 K0, SW23 K0, SW24 K0, SW25 K0, SW26 K0, SW27 K0, SW28 K0, SW29 K0, SW3 K0, SW30 K0, SW31 K0, SW32 K0, SW33 K0, SW34 K0, SW35 K0, SW36 K0, SW37 K0, SW38 K0, SW39 K0, SW4 K0, SW40 K0, SW41 K0, SW42 K0, SW43 K0, SW44 K0, SW45 K0, SW46 K0, SW47 K0, SW48 K0, SW49 K0, SW5 K0, SW50 K0, SW51 K0, SW52 K0, SW53 K0, SW54 K0, SW55 K0, SW56 K0, SW57 K0, SW58 K0, SW59 K0, SW6 K0, SW60 K0, SW61 K0, SW62 K0, SW63 K0, SW64 K0, SW65 K0, SW66 K0, SW67 K0, SW68 K0, SW69 K0, SW7 K0, SW70 K0, SW71 K0, SW72 K0, SW73 K0, SW74 K0, SW75 K0, SW76 K0, SW77 K0, SW78 K0, SW79 K0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

Commit message: continue working on routing added a second 2u bs compat
Parts:
- added SW14.5: K0, keebrary_mx:MX_PCB_200H, F.Cu at (490.5, 157.2)
- SW14: footprint wood_kailh_socket:Kailh_MX_Socket -> keebrary_mx:MX_PCB_100H; moved to F.Cu
- SW15, SW17, SW78: footprint ai03_hybrid:MX-1U-NoLED -> keebrary_mx:MX_PCB_100H
- SW16: footprint ai03_hybrid:MX-2U-NoLED -> keebrary_mx:MX_PCB_200H
- moved R2 21.0 mm to (238.8, 156.5)
- moved R1 20.5 mm to (242.6, 156.5)
- moved P1 4.70 mm to (245.3, 223.8), turned to 90 degrees
- moved U1 4.27 mm to (245.9, 204.0), turned to 0 degrees
- moved C2 1.41 mm to (241.2, 178.6), turned to 180 degrees
- moved C1 0.67 mm to (241.2, 172.8)
- turned SW14 to 0 degrees
Connections:
- SW13 pad 1: /KEY13 -> GND
- SW13 pad 2: GND -> /KEY13
- SW14 pad 1: /KEY14 -> GND
- SW14 pad 2: GND -> /KEY14
- SW15 pad 1: /KEY15 -> GND
- SW15 pad 2: GND -> /KEY14.5
- SW16 pad 1: /KEY16 -> GND
- SW16 pad 2: GND -> /KEY16
- SW17 pad 1: /KEY17 -> /KEY16
- U1 pad 10: Net-(U1-Pad10) -> /KEY5
- U1 pad 11: Net-(U1-Pad11) -> /KEY6
- U1 pad 12: Net-(U1-Pad12) -> /KEY7
- U1 pad 15: Net-(U1-Pad15) -> /KEY8
- U1 pad 16: Net-(U1-Pad16) -> /KEY9
- U1 pad 17: Net-(U1-Pad17) -> /KEY10
- U1 pad 18: Net-(U1-Pad18) -> /KEY11
- U1 pad 19: Net-(U1-Pad19) -> /KEY12
- U1 pad 20: Net-(U1-Pad20) -> /KEY13
- U1 pad 21: Net-(U1-Pad21) -> /KEY14
- U1 pad 22: Net-(U1-Pad22) -> /KEY14.5
- U1 pad 25: Net-(U1-Pad25) -> /KEY16
- U1 pad 26: Net-(U1-Pad26) -> /KEY18
- U1 pad 7: Net-(U1-Pad7) -> /KEY2
- U1 pad 8: Net-(U1-Pad8) -> /KEY3
- U1 pad 9: Net-(U1-Pad9) -> /KEY4
Routing:
- net GND: track 0.00 -> 152.8 mm, vias 0 -> 10
- net VCC: track 0.00 -> 135.7 mm
- net /KEY0: track 77.8 -> 0.00 mm
- net /KEY1: track 67.9 -> 0.00 mm
- net /KEY19: track 58.7 -> 0.00 mm
- net Net-(J1-PadA7): track 0.00 -> 57.0 mm
- net Net-(J1-PadA6): track 0.00 -> 55.5 mm
- net /KEY68: track 54.5 -> 0.00 mm
- net /KEY20: track 48.9 -> 0.00 mm
- net /KEY36: track 46.2 -> 0.00 mm
- net /KEY69: track 40.4 -> 0.00 mm
- net /KEY52: track 37.8 -> 0.00 mm
- net +5V: track 0.00 -> 35.0 mm, vias 0 -> 2
- net /KEY37: track 27.8 -> 0.00 mm
- net /KEY53: track 19.7 -> 0.00 mm
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