File: 65plus/65_plus/65_plus.sch (KiCad schematic (older format))
At the start: 91 parts, among them J1 USB_Type_C_2.0_Receptacle, P1 TC2030-IDC, SW0 K0, SW1 K0, SW10 K0, SW11 K0, SW12 K0, SW13 K0, SW14 K0, SW15 K0, SW16 K0, SW17 K0, SW18 K0, SW19 K0, SW2 K0, SW20 K0, SW21 K0, SW22 K0, SW23 K0, SW24 K0, SW25 K0, SW26 K0, SW27 K0, SW28 K0, SW29 K0, SW3 K0, SW30 K0, SW31 K0, SW32 K0, SW33 K0, SW34 K0, SW35 K0, SW36 K0, SW37 K0, SW38 K0, SW39 K0, SW4 K0, SW40 K0, SW41 K0, SW42 K0, SW43 K0, SW44 K0, SW45 K0, SW46 K0, SW47 K0, SW48 K0, SW49 K0, SW5 K0, SW50 K0, SW51 K0, SW52 K0, SW53 K0, SW54 K0, SW55 K0, SW56 K0, SW57 K0, SW58 K0, SW59 K0, SW6 K0, SW60 K0, SW61 K0, SW62 K0, SW63 K0, SW64 K0, SW65 K0, SW66 K0, SW67 K0, SW68 K0, SW69 K0, SW7 K0, SW70 K0, SW71 K0, SW72 K0, SW73 K0, SW74 K0, SW75 K0, SW76 K0, SW77 K0, SW78 K0, SW79 K0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

Commit message: continue working on routing added a second 2u bs compat
Parts:
- added SW14.5: K0, keebrary_mx:MX_PCB_200H, symbol keyboard_parts:SW_PUSH
- SW14: footprint wood_kailh_socket:Kailh_MX_Socket -> keebrary_mx:MX_PCB_100H
- SW15, SW17, SW78: footprint ai03_hybrid:MX-1U-NoLED -> keebrary_mx:MX_PCB_100H
- SW16: footprint ai03_hybrid:MX-2U-NoLED -> keebrary_mx:MX_PCB_200H
Connections:
- net labels added: KEY14.5
- wire segments 145 -> 154
Changed lines of the file:
@@
 F 3 "" H 2000 6150 60  0000 C CNN
 	1    2000 6150
-	1    0    0    -1
+	-1   0    0    -1
 $EndComp
 $Comp
@@
 F 0 "SW14" H 2000 6655 50  0000 C CNN
 F 1 "K0" H 2000 6564 50  0000 C CNN
-F 2 "wood_kailh_socket:Kailh_MX_Socket" H 2000 6400 60  0001 C CNN
+F 2 "keebrary_mx:MX_PCB_100H" H 2000 6400 60  0001 C CNN
 F 3 "" H 2000 6400 60  0000 C CNN
 	1    2000 6400
-	1    0    0    -1
+	-1   0    0    -1
 $EndComp
 $Comp
@@
 F 0 "SW15" H 2000 6955 50  0000 C CNN
 F 1 "K0" H 2000 6864 50  0000 C CNN
-F 2 "ai03_hybrid:MX-1U-NoLED" H 2000 6700 60  0001 C CNN
+F 2 "keebrary_mx:MX_PCB_100H" H 2000 6700 60  0001 C CNN
 F 3 "" H 2000 6700 60  0000 C CNN
 	1    2000 6700
-	1    0    0    -1
+	-1   0    0    -1
 $EndComp
 $Comp
@@
 F 0 "SW16" H 2000 7205 50  0000 C CNN
 F 1 "K0" H 2000 7114 50  0000 C CNN
-F 2 "ai03_hybrid:MX-2U-NoLED" H 2000 6950 60  0001 C CNN
+F 2 "keebrary_mx:MX_PCB_200H" H 2000 6950 60  0001 C CNN
 F 3 "" H 2000 6950 60  0000 C CNN
 	1    2000 6950
-	1    0    0    -1
+	-1   0    0    -1
 $EndComp
 $Comp
@@
 F 0 "SW17" H 2000 7505 50  0000 C CNN
 F 1 "K0" H 2000 7414 50  0000 C CNN
-F 2 "ai03_hybrid:MX-1U-NoLED" H 2000 7250 60  0001 C CNN
+F 2 "keebrary_mx:MX_PCB_100H" H 2000 7250 60  0001 C CNN
 F 3 "" H 2000 7250 60  0000 C CNN
 	1    2000 7250
@@
 F 0 "SW78" H 6550 7805 50  0000 C CNN
 F 1 "K0" H 6550 7714 50  0000 C CNN
-F 2 "ai03_hybrid:MX-1U-NoLED" H 6550 7550 60  0001 C CNN
+F 2 "keebrary_mx:MX_PCB_100H" H 6550 7550 60  0001 C CNN
 F 3 "" H 6550 7550 60  0000 C CNN
 	1    6550 7550
@@
 KEY82
 Wire Wire Line
-	8150 5950 8150 6550
+	8150 5950 8150 6200
 $Comp
 L Device:C C2
@@
 Text Label 10450 4700 2    50   ~ 0
 KEY37
+Connection ~ 8150 6200
+Wire Wire Line
+	8150 6200 8150 6550
+$Comp
+L keyboard_parts:SW_PUSH SW14.5
+U 1 1 5B1E0FF7
+P 7850 6200
+F 0 "SW14.5" H 7850 6455 50  0000 C CNN
+F 1 "K0" H 7850 6364 50  0000 C CNN
+F 2 "keebrary_mx:MX_PCB_200H" H 7850 6200 60  0001 C CNN
+F 3 "" H 7850 6200 60  0000 C CNN
+	1    7850 6200
+	-1   0    0    -1
+$EndComp
+Text Label 7550 6200 2    50   ~ 0
+KEY14.5
+Text Label 10450 4900 2    50   ~ 0
+KEY3
+Text Label 10450 5000 2    50   ~ 0
+KEY4
+Text Label 10450 5100 2    50   ~ 0
+KEY5
+Text Label 10450 5200 2    50   ~ 0
+KEY6
+Text Label 10450 5300 2    50   ~ 0
+KEY7
+Text Label 10450 5450 2    50   ~ 0
+KEY8
+Text Label 10450 5550 2    50   ~ 0
+KEY9
+Text Label 10450 5650 2    50   ~ 0
+KEY10
+Text Label 10450 5750 2    50   ~ 0
+KEY11
+Text Label 10450 5850 2    50   ~ 0
+KEY12
+Text Label 10450 5950 2    50   ~ 0
+KEY13
+Text Label 10450 6050 2    50   ~ 0
+KEY14
+Text Label 10200 6150 2    50   ~ 0
+KEY15
+Text Label 10200 6250 2    50   ~ 0
+KEY16
+Text Label 10200 6300 2    50   ~ 0
+KEY17
+Text Label 10450 6400 2    50   ~ 0
+KEY18
+Text Label 10200 6100 2    50   ~ 0
+KEY14.5
+Text Label 10450 4800 2    50   ~ 0
+KEY2
+Wire Wire Line
+	10200 6100 10250 6100
+Wire Wire Line
+	10250 6100 10250 6150
+Wire Wire Line
+	10250 6150 10200 6150
+Wire Wire Line
+	10250 6150 10450 6150
+Connection ~ 10250 6150
+Wire Wire Line
+	10200 6250 10250 6250
+Wire Wire Line
+	10250 6250 10250 6300
+Wire Wire Line
+	10250 6300 10200 6300
+Wire Wire Line
+	10250 6300 10450 6300
+Connection ~ 10250 6300
 $EndSCHEMATC
