File: 65plus/65_plus_PIN_GND/65_plus.kicad_pcb (KiCad board)
At the start: 2 copper layers, 352.4 x 104.8 mm, 92 parts, among them J1 USB_Type_C_2.0_Receptacle, P1 TC2030-IDC, SW0 K0, SW1 K0, SW10 K0, SW11 K0, SW12 K0, SW13 K0, SW14 K0, SW14.5 K0, SW15 K0, SW16 K0, SW17 K0, SW18 K0, SW19 K0, SW2 K0, SW20 K0, SW21 K0, SW22 K0, SW23 K0, SW24 K0, SW25 K0, SW26 K0, SW27 K0, SW28 K0, SW29 K0, SW3 K0, SW30 K0, SW31 K0, SW32 K0, SW33 K0, SW34 K0, SW35 K0, SW36 K0, SW37 K0, SW38 K0, SW39 K0, SW4 K0, SW40 K0, SW41 K0, SW42 K0, SW43 K0, SW44 K0, SW45 K0, SW46 K0, SW47 K0, SW48 K0, SW49 K0, SW5 K0, SW50 K0, SW51 K0, SW52 K0, SW53 K0, SW54 K0, SW55 K0, SW56 K0, SW57 K0, SW58 K0, SW59 K0, SW6 K0, SW60 K0, SW61 K0, SW62 K0, SW63 K0, SW64 K0, SW65 K0, SW66 K0, SW67 K0, SW68 K0, SW69 K0, SW7 K0, SW70 K0, SW71 K0, SW72 K0, SW73 K0, SW74 K0, SW75 K0, SW76 K0, SW77 K0, SW78 K0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

Commit message: 90 plus almost complete
Parts:
- removed SW18, SW71: K0, wood_kailh_socket:Kailh_MX_Socket
- removed SW73, SW76, SW77: K0, ai03_hybrid:MX-3U-ReversedStabilizers-NoLED
- SW14, SW15, SW17, SW78: footprint keebrary_mx:MX_PCB_100H -> ai03_hybrid:MX-1U-NoLED
- SW14.5, SW16: footprint keebrary_mx:MX_PCB_200H -> ai03_hybrid:MX-2U-NoLED
- SW74: footprint ai03_hybrid:MX-7U-ReversedStabilizers-NoLED -> ai03_hybrid:MX-7U-NoLED
- SW75: footprint ai03_hybrid:MX-6U-7UOverlay-ReversedStabilizers -> ai03_hybrid:MX-6U-7UOverlay
Connections:
- SW0 pad 1: /KEY0 -> GND
- SW0 pad 2: GND -> /KEY0
- SW13 pad 1: GND -> /KEY13
- SW13 pad 2: /KEY13 -> GND
- SW14 pad 1: GND -> /KEY14
- SW14 pad 2: /KEY14 -> GND
- SW14.5 pad 1: GND -> /KEY14.5
- SW14.5 pad 2: /KEY14.5 -> GND
- SW15 pad 1: GND -> /KEY14.5
- SW15 pad 2: /KEY14.5 -> GND
- SW16 pad 1: GND -> /KEY16
- SW16 pad 2: /KEY16 -> GND
- SW19 pad 1: /KEY19 -> GND
- SW19 pad 2: GND -> /KEY19
- SW36 pad 1: /KEY36 -> GND
- SW36 pad 2: GND -> /KEY36
- SW38 pad 1: /KEY38 -> GND
- SW38 pad 2: GND -> /KEY38
- SW52 pad 1: /KEY52 -> GND
- SW52 pad 2: GND -> /KEY52
- SW68 pad 1: /KEY68 -> GND
- SW68 pad 2: GND -> /KEY68
- U1 pad 1: /KEY0 -> /KEY53
- U1 pad 10: /KEY5 -> /KEY1
- U1 pad 100: /KEY19 -> /KEY80
- U1 pad 11: /KEY6 -> /KEY20
- U1 pad 12: /KEY7 -> /KEY37
- U1 pad 15: /KEY8 -> /KEY2
- U1 pad 16: /KEY9 -> /KEY3
- U1 pad 17: /KEY10 -> /KEY4
- U1 pad 18: /KEY11 -> /KEY5
- U1 pad 19: /KEY12 -> /KEY6
- U1 pad 2: /KEY1 -> /KEY69
- U1 pad 20: /KEY13 -> /KEY7
- U1 pad 21: /KEY14 -> /KEY8
- U1 pad 22: /KEY14.5 -> /KEY9
- U1 pad 25: /KEY16 -> /KEY10
- U1 pad 26: /KEY18 -> /KEY11
- U1 pad 27: Net-(U1-Pad27) -> /KEY12
- U1 pad 28: Net-(U1-Pad28) -> /KEY13
- U1 pad 29: Net-(U1-Pad29) -> /KEY14
- U1 pad 30: Net-(U1-Pad30) -> /KEY14.5
- U1 pad 35: Net-(U1-Pad35) -> /KEY16
- U1 pad 36: Net-(U1-Pad36) -> /KEY54
- U1 pad 37: Net-(U1-Pad37) -> /KEY21
- U1 pad 38: Net-(U1-Pad38) -> /KEY22
- U1 pad 39: Net-(U1-Pad39) -> /KEY23
- U1 pad 40: Net-(U1-Pad40) -> /KEY24
- U1 pad 41: Net-(U1-Pad41) -> /KEY25
- U1 pad 42: Net-(U1-Pad42) -> /KEY26
- U1 pad 45: Net-(U1-Pad45) -> /KEY82
- U1 pad 46: Net-(U1-Pad46) -> /KEY81
- U1 pad 47: Net-(U1-Pad47) -> /KEY27
- U1 pad 48: Net-(U1-Pad48) -> /KEY28
- U1 pad 49: Net-(U1-Pad49) -> /KEY29
- U1 pad 5: /KEY20 -> /KEY68
- U1 pad 50: Net-(U1-Pad50) -> /KEY30
- U1 pad 51: Net-(U1-Pad51) -> /KEY31
- U1 pad 52: Net-(U1-Pad52) -> /KEY32
- U1 pad 55: Net-(U1-Pad55) -> /KEY33
- U1 pad 56: Net-(U1-Pad56) -> /KEY34
- U1 pad 57: Net-(U1-Pad57) -> /KEY35
- U1 pad 58: Net-(U1-Pad58) -> /KEY38
- U1 pad 59: Net-(U1-Pad59) -> /KEY39
- U1 pad 6: /KEY37 -> /KEY52
- U1 pad 60: Net-(U1-Pad60) -> /KEY40
- U1 pad 61: Net-(U1-Pad61) -> /KEY41
- U1 pad 62: Net-(U1-Pad62) -> /KEY42
- U1 pad 65: Net-(U1-Pad65) -> /KEY43
- U1 pad 66: Net-(U1-Pad66) -> /KEY44
- U1 pad 67: Net-(U1-Pad67) -> /KEY45
- U1 pad 68: Net-(U1-Pad68) -> /KEY46
- U1 pad 69: Net-(U1-Pad69) -> /KEY47
- U1 pad 7: /KEY2 -> /KEY36
- U1 pad 70: Net-(U1-Pad70) -> /KEY48
- U1 pad 71: Net-(U1-Pad71) -> /KEY49
- U1 pad 72: Net-(U1-Pad72) -> /KEY50
- U1 pad 75: Net-(U1-Pad75) -> /KEY51
- U1 pad 76: Net-(U1-Pad76) -> /KEY55
- U1 pad 77: Net-(U1-Pad77) -> /KEY56
- U1 pad 78: Net-(U1-Pad78) -> /KEY57
- U1 pad 79: Net-(U1-Pad79) -> /KEY58
- U1 pad 8: /KEY3 -> /KEY19
- U1 pad 80: Net-(U1-Pad80) -> /KEY59
- U1 pad 81: Net-(U1-Pad81) -> /KEY60
- U1 pad 82: Net-(U1-Pad82) -> /KEY61
- U1 pad 85: Net-(U1-Pad85) -> /KEY62
- U1 pad 86: Net-(U1-Pad86) -> /KEY63
- U1 pad 87: Net-(U1-Pad87) -> /KEY64
- U1 pad 88: Net-(U1-Pad88) -> /KEY65
- U1 pad 9: /KEY4 -> /KEY0
- U1 pad 91: Net-(U1-Pad91) -> /KEY66
- U1 pad 92: Net-(U1-Pad92) -> /KEY67
- U1 pad 95: /KEY53 -> /KEY70
- U1 pad 96: /KEY69 -> /KEY72
- U1 pad 97: /KEY68 -> /KEY74
- U1 pad 98: /KEY52 -> /KEY78
- U1 pad 99: /KEY36 -> /KEY79
Routing:
- net /KEY82: track 0.00 -> 339.2 mm, vias 0 -> 4
- net /KEY81: track 0.00 -> 321.2 mm, vias 0 -> 4
- net /KEY16: track 0.00 -> 314.3 mm, vias 0 -> 1
- net /KEY67: track 0.00 -> 312.4 mm
- net /KEY66: track 0.00 -> 292.5 mm
- net /KEY14.5: track 0.00 -> 292.4 mm, vias 0 -> 1
- net /KEY35: track 0.00 -> 288.6 mm
- net /KEY51: track 0.00 -> 284.5 mm
- net /KEY80: track 0.00 -> 277.9 mm
- net /KEY14: track 0.00 -> 270.0 mm, vias 0 -> 1
- net /KEY34: track 0.00 -> 264.6 mm
- net /KEY50: track 0.00 -> 252.8 mm
- net /KEY65: track 0.00 -> 252.2 mm, vias 0 -> 2
- net /KEY13: track 0.00 -> 251.2 mm, vias 0 -> 2
- net /KEY79: track 0.00 -> 243.6 mm
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