File: 65plus/65_plus_PIN_GND/65_plus.sch (KiCad schematic (older format))
At the start: 92 parts, among them J1 USB_Type_C_2.0_Receptacle, P1 TC2030-IDC, SW0 K0, SW1 K0, SW10 K0, SW11 K0, SW12 K0, SW13 K0, SW14 K0, SW14.5 K0, SW15 K0, SW16 K0, SW17 K0, SW18 K0, SW19 K0, SW2 K0, SW20 K0, SW21 K0, SW22 K0, SW23 K0, SW24 K0, SW25 K0, SW26 K0, SW27 K0, SW28 K0, SW29 K0, SW3 K0, SW30 K0, SW31 K0, SW32 K0, SW33 K0, SW34 K0, SW35 K0, SW36 K0, SW37 K0, SW38 K0, SW39 K0, SW4 K0, SW40 K0, SW41 K0, SW42 K0, SW43 K0, SW44 K0, SW45 K0, SW46 K0, SW47 K0, SW48 K0, SW49 K0, SW5 K0, SW50 K0, SW51 K0, SW52 K0, SW53 K0, SW54 K0, SW55 K0, SW56 K0, SW57 K0, SW58 K0, SW59 K0, SW6 K0, SW60 K0, SW61 K0, SW62 K0, SW63 K0, SW64 K0, SW65 K0, SW66 K0, SW67 K0, SW68 K0, SW69 K0, SW7 K0, SW70 K0, SW71 K0, SW72 K0, SW73 K0, SW74 K0, SW75 K0, SW76 K0, SW77 K0, SW78 K0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

Commit message: 90 plus almost complete
Parts:
- SW14, SW15, SW17, SW78: footprint keebrary_mx:MX_PCB_100H -> ai03_hybrid:MX-1U-NoLED
- SW14.5, SW16: footprint keebrary_mx:MX_PCB_200H -> ai03_hybrid:MX-2U-NoLED
- SW73, SW76, SW77: footprint ai03_hybrid:MX-3U-ReversedStabilizers-NoLED -> ai03_hybrid:MX-3U-NoLED
- SW74: footprint ai03_hybrid:MX-7U-ReversedStabilizers-NoLED -> ai03_hybrid:MX-7U-NoLED
- SW75: footprint ai03_hybrid:MX-6U-7UOverlay-ReversedStabilizers -> ai03_hybrid:MX-6U-7UOverlay
Changed lines of the file:
@@
 EESchema Schematic File Version 4
+LIBS:65_plus-cache
 EELAYER 26 0
 EELAYER END
@@
 F 3 "" H 2000 1700 60  0000 C CNN
 	1    2000 1700
-	1    0    0    -1
+	-1   0    0    -1
 $EndComp
 $Comp
@@
 F 3 "" H 6550 3950 60  0000 C CNN
 	1    6550 3950
-	1    0    0    -1
+	-1   0    0    -1
 $EndComp
 $Comp
@@
 F 3 "" H 2000 6150 60  0000 C CNN
 	1    2000 6150
-	-1   0    0    -1
+	1    0    0    -1
 $EndComp
 $Comp
@@
 F 0 "SW14" H 2000 6655 50  0000 C CNN
 F 1 "K0" H 2000 6564 50  0000 C CNN
-F 2 "keebrary_mx:MX_PCB_100H" H 2000 6400 60  0001 C CNN
+F 2 "ai03_hybrid:MX-1U-NoLED" H 2000 6400 60  0001 C CNN
 F 3 "" H 2000 6400 60  0000 C CNN
 	1    2000 6400
-	-1   0    0    -1
+	1    0    0    -1
 $EndComp
 $Comp
@@
 F 0 "SW15" H 2000 6955 50  0000 C CNN
 F 1 "K0" H 2000 6864 50  0000 C CNN
-F 2 "keebrary_mx:MX_PCB_100H" H 2000 6700 60  0001 C CNN
+F 2 "ai03_hybrid:MX-1U-NoLED" H 2000 6700 60  0001 C CNN
 F 3 "" H 2000 6700 60  0000 C CNN
 	1    2000 6700
-	-1   0    0    -1
+	1    0    0    -1
 $EndComp
 $Comp
@@
 F 0 "SW16" H 2000 7205 50  0000 C CNN
 F 1 "K0" H 2000 7114 50  0000 C CNN
-F 2 "keebrary_mx:MX_PCB_200H" H 2000 6950 60  0001 C CNN
+F 2 "ai03_hybrid:MX-2U-NoLED" H 2000 6950 60  0001 C CNN
 F 3 "" H 2000 6950 60  0000 C CNN
 	1    2000 6950
-	-1   0    0    -1
+	1    0    0    -1
 $EndComp
 $Comp
@@
 F 0 "SW17" H 2000 7505 50  0000 C CNN
 F 1 "K0" H 2000 7414 50  0000 C CNN
-F 2 "keebrary_mx:MX_PCB_100H" H 2000 7250 60  0001 C CNN
+F 2 "ai03_hybrid:MX-1U-NoLED" H 2000 7250 60  0001 C CNN
 F 3 "" H 2000 7250 60  0000 C CNN
 	1    2000 7250
@@
 F 3 "" H 2000 7850 60  0000 C CNN
 	1    2000 7850
-	1    0    0    -1
+	-1   0    0    -1
 $EndComp
 $Comp
@@
 F 3 "" H 3600 6950 60  0000 C CNN
 	1    3600 6950
-	1    0    0    -1
+	-1   0    0    -1
 $EndComp
 $Comp
@@
 F 3 "" H 3600 7550 60  0000 C CNN
 	1    3600 7550
-	1    0    0    -1
+	-1   0    0    -1
 $EndComp
 $Comp
@@
 F 3 "" H 4950 5850 60  0000 C CNN
 	1    4950 5850
-	1    0    0    -1
+	-1   0    0    -1
 $EndComp
 $Comp
@@
 F 0 "SW73" H 6550 6405 50  0000 C CNN
 F 1 "K0" H 6550 6314 50  0000 C CNN
-F 2 "ai03_hybrid:MX-3U-ReversedStabilizers-NoLED" H 6550 6150 60  0001 C CNN
+F 2 "ai03_hybrid:MX-3U-NoLED" H 6550 6150 60  0001 C CNN
 F 3 "" H 6550 6150 60  0000 C CNN
 	1    6550 6150
@@
 F 0 "SW74" H 6550 6705 50  0000 C CNN
 F 1 "K0" H 6550 6614 50  0000 C CNN
-F 2 "ai03_hybrid:MX-7U-ReversedStabilizers-NoLED" H 6550 6450 60  0001 C CNN
+F 2 "ai03_hybrid:MX-7U-NoLED" H 6550 6450 60  0001 C CNN
 F 3 "" H 6550 6450 60  0000 C CNN
 	1    6550 6450
@@
 F 0 "SW75" H 6550 7005 50  0000 C CNN
 F 1 "K0" H 6550 6914 50  0000 C CNN
-F 2 "ai03_hybrid:MX-6U-7UOverlay-ReversedStabilizers" H 6550 6750 60  0001 C CNN
+F 2 "ai03_hybrid:MX-6U-7UOverlay" H 6550 6750 60  0001 C CNN
 F 3 "" H 6550 6750 60  0000 C CNN
 	1    6550 6750
@@
 F 0 "SW76" H 6550 7255 50  0000 C CNN
 F 1 "K0" H 6550 7164 50  0000 C CNN
-F 2 "ai03_hybrid:MX-3U-ReversedStabilizers-NoLED" H 6550 7000 60  0001 C CNN
+F 2 "ai03_hybrid:MX-3U-NoLED" H 6550 7000 60  0001 C CNN
 F 3 "" H 6550 7000 60  0000 C CNN
 	1    6550 7000
@@
 F 0 "SW77" H 6550 7555 50  0000 C CNN
 F 1 "K0" H 6550 7464 50  0000 C CNN
-F 2 "ai03_hybrid:MX-3U-ReversedStabilizers-NoLED" H 6550 7300 60  0001 C CNN
+F 2 "ai03_hybrid:MX-3U-NoLED" H 6550 7300 60  0001 C CNN
 F 3 "" H 6550 7300 60  0000 C CNN
 	1    6550 7300
@@
 F 0 "SW78" H 6550 7805 50  0000 C CNN
 F 1 "K0" H 6550 7714 50  0000 C CNN
-F 2 "keebrary_mx:MX_PCB_100H" H 6550 7550 60  0001 C CNN
+F 2 "ai03_hybrid:MX-1U-NoLED" H 6550 7550 60  0001 C CNN
 F 3 "" H 6550 7550 60  0000 C CNN
 	1    6550 7550
@@
 Wire Wire Line
 	12000 3000 12000 3450
-Text Label 10450 3750 2    50   ~ 0
+Text Label 10450 4350 2    50   ~ 0
 KEY53
-Text Label 10450 3850 2    50   ~ 0
+Text Label 10450 4450 2    50   ~ 0
 KEY69
-Text Label 10450 3950 2    50   ~ 0
+Text Label 10450 4600 2    50   ~ 0
 KEY68
-Text Label 10450 4050 2    50   ~ 0
+Text Label 10450 4700 2    50   ~ 0
 KEY52
-Text Label 10450 4150 2    50   ~ 0
+Text Label 10450 4800 2    50   ~ 0
 KEY36
-Text Label 10450 4250 2    50   ~ 0
+Text Label 10450 4900 2    50   ~ 0
 KEY19
-Text Label 10450 4350 2    50   ~ 0
+Text Label 10450 5000 2    50   ~ 0
 KEY0
-Text Label 10450 4450 2    50   ~ 0
+Text Label 10450 5100 2    50   ~ 0
 KEY1
-Text Label 10450 4600 2    50   ~ 0
+Text Label 10450 5200 2    50   ~ 0
 KEY20
-Text Label 10450 4700 2    50   ~ 0
+Text Label 10450 5300 2    50   ~ 0
 KEY37
 Connection ~ 8150 6200
@@
 F 0 "SW14.5" H 7850 6455 50  0000 C CNN
 F 1 "K0" H 7850 6364 50  0000 C CNN
-F 2 "keebrary_mx:MX_PCB_200H" H 7850 6200 60  0001 C CNN
+F 2 "ai03_hybrid:MX-2U-NoLED" H 7850 6200 60  0001 C CNN
 F 3 "" H 7850 6200 60  0000 C CNN
 	1    7850 6200
-	-1   0    0    -1
+	1    0    0    -1
 $EndComp
 Text Label 7550 6200 2    50   ~ 0
 KEY14.5
-Text Label 10450 4900 2    50   ~ 0
+Text Label 10450 5550 2    50   ~ 0
 KEY3
-Text Label 10450 5000 2    50   ~ 0
+Text Label 10450 5650 2    50   ~ 0
 KEY4
-Text Label 10450 5100 2    50   ~ 0
+Text Label 10450 5750 2    50   ~ 0
 KEY5
-Text Label 10450 5200 2    50   ~ 0
+Text Label 10450 5850 2    50   ~ 0
 KEY6
-Text Label 10450 5300 2    50   ~ 0
+Text Label 10450 5950 2    50   ~ 0
 KEY7
+Text Label 10450 6050 2    50   ~ 0
+KEY8
+Text Label 10450 6150 2    50   ~ 0
+KEY9
+Text Label 10450 6300 2    50   ~ 0
+KEY10
+Text Label 10450 6400 2    50   ~ 0
+KEY11
+Text Label 10450 6500 2    50   ~ 0
+KEY12
+Text Label 10450 6600 2    50   ~ 0
+KEY13
+Text Label 10450 6700 2    50   ~ 0
+KEY14
+Text Label 10200 6800 2    50   ~ 0
+KEY15
+Text Label 10200 7100 2    50   ~ 0
+KEY16
+Text Label 10200 7150 2    50   ~ 0
+KEY17
+Text Label 10200 6750 2    50   ~ 0
+KEY14.5
 Text Label 10450 5450 2    50   ~ 0
-KEY8
-Text Label 10450 5550 2    50   ~ 0
-KEY9
-Text Label 10450 5650 2    50   ~ 0
-KEY10
-Text Label 10450 5750 2    50   ~ 0
-KEY11
-Text Label 10450 5850 2    50   ~ 0
-KEY12
-Text Label 10450 5950 2    50   ~ 0
-KEY13
-Text Label 10450 6050 2    50   ~ 0
-KEY14
-Text Label 10200 6150 2    50   ~ 0
-KEY15
-Text Label 10200 6250 2    50   ~ 0
-KEY16
-Text Label 10200 6300 2    50   ~ 0
-KEY17
-Text Label 10450 6400 2    50   ~ 0
-KEY18
-Text Label 10200 6100 2    50   ~ 0
-KEY14.5
-Text Label 10450 4800 2    50   ~ 0
 KEY2
 Wire Wire Line
-	10200 6100 10250 6100
-Wire Wire Line
-	10250 6100 10250 6150
-Wire Wire Line
-	10250 6150 10200 6150
-Wire Wire Line
-	10250 6150 10450 6150
-Connection ~ 10250 6150
-Wire Wire Line
-	10200 6250 10250 6250
-Wire Wire Line
-	10250 6250 10250 6300
-Wire Wire Line
-	10250 6300 10200 6300
-Wire Wire Line
-	10250 6300 10450 6300
-Connection ~ 10250 6300
+	10200 6750 10250 6750
+Wire Wire Line
+	10250 6750 10250 6800
+Wire Wire Line
+	10250 6800 10200 6800
+Wire Wire Line
+	10250 6800 10450 6800
+Connection ~ 10250 6800
+Wire Wire Line
+	10200 7100 10250 7100
+Wire Wire Line
+	10250 7100 10250 7150
+Wire Wire Line
+	10250 7150 10200 7150
+Wire Wire Line
+	10250 7150 10450 7150
+Connection ~ 10250 7150
+Text Label 10450 7350 2    50   ~ 0
+KEY21
+Text Label 10450 7450 2    50   ~ 0
+KEY22
+Text Label 10450 7550 2    50   ~ 0
+KEY23
+Text Label 10450 7650 2    50   ~ 0
+KEY24
+Text Label 10450 7750 2    50   ~ 0
+KEY25
+Text Label 10450 7850 2    50   ~ 0
+KEY26
+Text Label 12850 7450 0    50   ~ 0
+KEY27
+Text Label 12850 7550 0    50   ~ 0
+KEY28
+Text Label 12850 7650 0    50   ~ 0
+KEY29
+Text Label 12850 7750 0    50   ~ 0
+KEY30
+Text Label 12850 7850 0    50   ~ 0
+KEY31
+Text Label 12850 7950 0    50   ~ 0
+KEY32
+Text Label 12850 6400 0    50   ~ 0
+KEY33
+Text Label 12850 6500 0    50   ~ 0
+KEY34
+Text Label 12850 6600 0    50   ~ 0
+KEY35
+Text Label 12850 6700 0    50   ~ 0
+KEY38
+Text Label 12850 6800 0    50   ~ 0
+KEY39
+Text Label 12850 6900 0    50   ~ 0
+KEY40
+Text Label 12850 7000 0    50   ~ 0
+KEY41
+Text Label 12850 7100 0    50   ~ 0
+KEY42
+Text Label 12850 5550 0    50   ~ 0
+KEY43
+Text Label 12850 5650 0    50   ~ 0
+KEY44
+Text Label 12850 5750 0    50   ~ 0
+KEY45
+Text Label 12850 5850 0    50   ~ 0
+KEY46
+Text Label 12850 5950 0    50   ~ 0
+KEY47
+Text Label 12850 6050 0    50   ~ 0
+KEY48
+Text Label 12850 6150 0    50   ~ 0
+KEY49
+Text Label 12850 6250 0    50   ~ 0
+KEY50
+Text Label 12850 4700 0    50   ~ 0
+KEY51
+Text Label 10450 7250 2    50   ~ 0
+KEY54
+Text Label 12850 4800 0    50   ~ 0
+KEY55
+Text Label 12850 4900 0    50   ~ 0
+KEY56
+Text Label 12850 5000 0    50   ~ 0
+KEY57
+Text Label 12850 5100 0    50   ~ 0
+KEY58
+Text Label 12850 5200 0    50   ~ 0
+KEY59
+Text Label 12850 5300 0    50   ~ 0
+KEY60
+Text Label 12850 5400 0    50   ~ 0
+KEY61
+Text Label 12850 4250 0    50   ~ 0
+KEY62
+Text Label 12850 4350 0    50   ~ 0
+KEY63
+Text Label 12850 4450 0    50   ~ 0
+KEY64
+Text Label 12850 4550 0    50   ~ 0
+KEY65
+Text Label 12850 4000 0    50   ~ 0
+KEY66
+Text Label 12850 4100 0    50   ~ 0
+KEY67
+Text Label 13450 7100 0    50   ~ 0
+KEY68
+Text Label 13450 7400 0    50   ~ 0
+KEY69
+Text Label 10450 3750 2    50   ~ 0
+KEY70
+Text Label 10450 3850 2    50   ~ 0
+KEY72
+Text Label 14600 5850 0    50   ~ 0
+KEY73
+Text Label 10450 3950 2    50   ~ 0
+KEY74
+Text Label 14600 6450 0    50   ~ 0
+KEY75
+Text Label 14600 6700 0    50   ~ 0
+KEY76
+Text Label 14600 7000 0    50   ~ 0
+KEY77
+Text Label 10450 4050 2    50   ~ 0
+KEY78
+Text Label 10450 4150 2    50   ~ 0
+KEY79
+Text Label 10450 4250 2    50   ~ 0
+KEY80
+Text Label 12850 7350 0    50   ~ 0
+KEY81
+Text Label 12850 7250 0    50   ~ 0
+KEY82
 $EndSCHEMATC
