File: 90plus/65plus_col2row/90plus_col2row.kicad_pcb (KiCad board)
At the start: 2 copper layers, 433.4 x 102.4 mm, 220 parts, among them J1 USB_Type_C_2.0_Receptacle, P1 TC2030-IDC, SW1 SW_PUSH, SW10 SW_PUSH, SW100 SW_PUSH, SW101 SW_PUSH, SW102 SW_PUSH, SW103 SW_PUSH, SW104 SW_PUSH, SW105 SW_PUSH, SW106 SW_PUSH, SW107 SW_PUSH, SW11 SW_PUSH, SW12 SW_PUSH, SW13 SW_PUSH, SW14 SW_PUSH, SW15 SW_PUSH, SW16 SW_PUSH, SW17 SW_PUSH, SW18 SW_PUSH, SW19 SW_PUSH, SW2 SW_PUSH, SW20 SW_PUSH, SW21 SW_PUSH, SW22 SW_PUSH, SW23 SW_PUSH, SW24 SW_PUSH, SW25 SW_PUSH, SW26 SW_PUSH, SW27 SW_PUSH, SW28 SW_PUSH, SW29 SW_PUSH, SW3 SW_PUSH, SW30 SW_PUSH, SW31 SW_PUSH, SW32 SW_PUSH, SW33 SW_PUSH, SW34 SW_PUSH, SW35 SW_PUSH, SW36 SW_PUSH, SW37 SW_PUSH, SW38 SW_PUSH, SW39 SW_PUSH, SW4 SW_PUSH, SW40 SW_PUSH, SW41 SW_PUSH, SW42 SW_PUSH, SW43 SW_PUSH, SW44 SW_PUSH, SW45 SW_PUSH, SW46 SW_PUSH, SW47 SW_PUSH, SW48 SW_PUSH, SW49 SW_PUSH, SW5 SW_PUSH, SW50 SW_PUSH, SW51 SW_PUSH, SW52 SW_PUSH, SW53 SW_PUSH, SW54 SW_PUSH, SW55 SW_PUSH, SW56 SW_PUSH, SW57 SW_PUSH, SW58 SW_PUSH, SW59 SW_PUSH, SW6 SW_PUSH, SW60 SW_PUSH, SW61 SW_PUSH, SW62 SW_PUSH, SW63 SW_PUSH, SW64 SW_PUSH, SW65 SW_PUSH, SW66 SW_PUSH, SW67 SW_PUSH, SW68 SW_PUSH, SW69 SW_PUSH, SW7 SW_PUSH, SW70 SW_PUSH, SW71 SW_PUSH, SW72 SW_PUSH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

Commit message: 90 plus complete TODO Cosmetics, R2 routing
Parts:
- added REF**: slot_10mm, Helpful:slot_10mm, F.Cu at (411.4, 323.2)
- added REF**: slot_10mm, Helpful:slot_10mm, F.Cu at (411.5, 233.7)
- moved REF** 2.97 mm to (411.6, 308.7)
- moved D93 2.39 mm to (419.1, 314.1)
- moved REF** 1.53 mm to (411.7, 279.5)
- moved REF** 0.59 mm to (411.6, 251.0)
Routing:
- net /ROW1: track 784.4 -> 710.5 mm
- net /COL21: track 497.6 -> 505.3 mm
- net /COL20: track 466.2 -> 473.0 mm
- net /ROW3: track 719.0 -> 722.7 mm
- net /ROW4: track 691.5 -> 694.3 mm
- net /PDI: track 45.9 -> 44.1 mm
- net Net-(D93-Pad2): track 5.74 -> 6.87 mm
- net /RST: track 43.6 -> 42.8 mm
