File: 100plus/project/Rev2/_autosave-100plus-2.kicad_pcb (KiCad board)
At the start: 2 copper layers, 433.4 x 121.4 mm, 279 parts, among them J1 USB_Type_C_2.0_Receptacle, K1 KEYSW, K10 KEYSW, K100 KEYSW, K101 KEYSW, K102 KEYSW, K103 KEYSW, K104 KEYSW, K105 KEYSW, K106 KEYSW, K107 KEYSW, K108 KEYSW, K109 KEYSW, K11 KEYSW, K110 KEYSW, K111 KEYSW, K112 KEYSW, K113 KEYSW, K114 KEYSW, K115 KEYSW, K116 KEYSW, K117 KEYSW, K118 KEYSW, K119 KEYSW, K12 KEYSW, K120 KEYSW, K121 KEYSW, K122 KEYSW, K123 KEYSW, K124 KEYSW, K125 KEYSW, K126 KEYSW, K127 KEYSW, K128 KEYSW, K129 KEYSW, K13 KEYSW, K130 KEYSW, K14 KEYSW, K15 KEYSW, K16 KEYSW, K17 KEYSW, K18 KEYSW, K19 KEYSW, K2 KEYSW, K20 KEYSW, K21 KEYSW, K22 KEYSW, K23 KEYSW, K24 KEYSW, K25 KEYSW, K26 KEYSW, K27 KEYSW, K28 KEYSW, K29 KEYSW, K3 KEYSW, K30 KEYSW, K31 KEYSW, K32 KEYSW, K33 KEYSW, K34 KEYSW, K35 KEYSW, K36 KEYSW, K37 KEYSW, K38 KEYSW, K39 KEYSW, K4 KEYSW, K40 KEYSW, K41 KEYSW, K42 KEYSW, K43 KEYSW, K44 KEYSW, K45 KEYSW, K46 KEYSW, K47 KEYSW, K48 KEYSW, K49 KEYSW, K5 KEYSW, K50 KEYSW, K51 KEYSW, K52 KEYSW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

Commit message: 100plus-2 is working
Parts:
- added B1: SPARKFUN_PRO_MICRO, SPARKFUN_PRO_MICRO, B.Cu at (435.8, 95.2)
- added REF**: slot_10mm, Helpful:slot_10mm, F.Cu at (95.5, 175.1)
- added REF**: slot_10mm, Helpful:slot_10mm, F.Cu at (95.4, 132.2)
- added REF**: slot_10mm, Helpful:slot_10mm, F.Cu at (95.5, 117.7)
- added REF**: mounting, wood_misc:mounting, F.Cu at (126.2, 138.1)
- added REF**: slot_10mm, Helpful:slot_10mm, F.Cu at (95.4, 147.2)
- added REF**: slot_10mm, Helpful:slot_10mm, F.Cu at (95.3, 74.9)
- added REF**: slot_10mm, Helpful:slot_10mm, F.Cu at (95.4, 160.9)
- added REF**: slot_10mm, Helpful:slot_10mm, F.Cu at (95.4, 103.6)
- added REF**: slot_10mm, Helpful:slot_10mm, F.Cu at (95.4, 89.5)
- moved R1 171.6 mm to (269.1, 83.3)
- moved P1 164.6 mm to (269.2, 102.7)
- moved U2 159.3 mm to (250.5, 98.3)
- moved C2 159.0 mm to (252.8, 85.1), turned to 90 degrees
- moved C1 155.6 mm to (250.2, 85.1), turned to 90 degrees
- moved J1 154.9 mm to (250.1, 72.4)
- moved U1 152.1 mm to (246.8, 84.8)
- moved R2 138.2 mm to (230.9, 83.5)
- moved D9 12.3 mm to (231.7, 97.0)
- moved D22 1.70 mm to (86.8, 114.3)
Connections:
- K10 pad 1: COL9 -> COL10
- K100 pad 1: COL11 -> COL13
- K101 pad 1: COL12 -> COL14
- K102 pad 1: COL14 -> COL16
- K103 pad 1: COL15 -> COL17
- K104 pad 1: COL16 -> COL18
- K105 pad 1: COL17 -> COL19
- K106 pad 1: COL18 -> COL20
- K107 pad 1: COL19 -> COL21
- K109 pad 1: COL19 -> COL21
- K11 pad 1: COL10 -> COL11
- K110 pad 1: COL9 -> COL10
- K115 pad 1: Net-(K115-Pad1) -> COL7
- K116 pad 1: COL9 -> COL10
- K117 pad 1: Net-(K117-Pad1) -> COL12
- K118 pad 1: COL11 -> COL13
- K119 pad 1: COL12 -> COL14
- K12 pad 1: COL11 -> COL13
- K120 pad 1: COL14 -> COL16
- K121 pad 1: COL15 -> COL17
- K122 pad 1: COL16 -> COL18
- K123 pad 1: COL17 -> COL19
- K124 pad 1: COL18 -> COL20
- K125 pad 1: COL19 -> COL21
- K127 pad 1: Net-(K117-Pad1) -> COL12
- K128 pad 1: COL16 -> COL18
- K129 pad 2: COL12 -> COL14
- K13 pad 1: COL12 -> COL14
- K14 pad 1: COL13 -> COL15
- K15 pad 1: COL14 -> COL16
- K16 pad 1: COL15 -> COL17
- K17 pad 1: COL16 -> COL18
- K18 pad 1: COL17 -> COL19
- K19 pad 1: COL18 -> COL20
- K20 pad 1: COL19 -> COL21
- K28 pad 1: Net-(K115-Pad1) -> COL7
- K29 pad 1: COL7 -> COL8
- K30 pad 1: COL8 -> COL9
- K31 pad 1: COL9 -> COL10
- K32 pad 1: COL10 -> COL11
- K33 pad 1: Net-(K117-Pad1) -> COL12
- K34 pad 1: COL11 -> COL13
- K35 pad 1: COL12 -> COL14
- K36 pad 1: COL13 -> COL15
- K37 pad 1: COL14 -> COL16
- K38 pad 1: COL15 -> COL17
- K39 pad 1: COL16 -> COL18
- K40 pad 1: COL17 -> COL19
- K41 pad 1: COL18 -> COL20
- K42 pad 1: COL19 -> COL21
- K43 pad 1: COL13 -> COL15
- K44 pad 1: COL14 -> COL16
- K52 pad 1: Net-(K115-Pad1) -> COL7
- K53 pad 1: COL7 -> COL8
- K54 pad 1: COL8 -> COL9
- K55 pad 1: COL9 -> COL10
- K56 pad 1: COL10 -> COL11
- K57 pad 1: Net-(K117-Pad1) -> COL12
- K58 pad 1: COL11 -> COL13
- K59 pad 1: COL12 -> COL14
- K60 pad 1: COL14 -> COL16
- K61 pad 1: COL15 -> COL17
- K62 pad 1: COL16 -> COL18
- K63 pad 1: COL17 -> COL19
- K64 pad 1: COL18 -> COL20
- K65 pad 1: COL19 -> COL21
- K66 pad 1: COL19 -> COL21
- K74 pad 1: Net-(K115-Pad1) -> COL7
- K75 pad 1: COL7 -> COL8
- K76 pad 1: COL8 -> COL9
- K77 pad 1: COL9 -> COL10
- K78 pad 1: COL10 -> COL11
- K79 pad 1: Net-(K117-Pad1) -> COL12
- K8 pad 1: COL7 -> COL8
- K80 pad 1: COL11 -> COL13
- K81 pad 1: COL12 -> COL14
- K82 pad 1: COL15 -> COL17
- K83 pad 1: COL16 -> COL18
- K84 pad 1: COL17 -> COL19
- K85 pad 1: COL18 -> COL20
- K86 pad 1: COL19 -> COL21
- K9 pad 1: COL8 -> COL9
- K94 pad 1: Net-(K115-Pad1) -> COL7
- K95 pad 1: COL7 -> COL8
- K96 pad 1: COL8 -> COL9
- K97 pad 1: COL9 -> COL10
- K98 pad 1: COL10 -> COL11
- K99 pad 1: Net-(K117-Pad1) -> COL12
- U2 pad 1: COL10 -> COL17
- U2 pad 10: COL18 -> ROW5
- U2 pad 11: COL19 -> ROW0
- U2 pad 12: Net-(U2-Pad12) -> COL5
- U2 pad 13: COL1 -> COL6
- U2 pad 14: ROW3 -> COL7
- U2 pad 15: ROW4 -> COL8
- U2 pad 16: ROW5 -> COL4
- U2 pad 17: COL0 -> COL3
- U2 pad 2: COL11 -> COL18
- U2 pad 20: ROW2 -> COL2
- U2 pad 21: ROW0 -> COL1
- U2 pad 22: ROW1 -> COL0
- U2 pad 23: COL3 -> Net-(U2-Pad23)
- U2 pad 24: COL4 -> Net-(U2-Pad24)
- U2 pad 25: Net-(U2-Pad25) -> COL21
- U2 pad 3: COL12 -> COL19
- U2 pad 32: COL2 -> COL20
- U2 pad 33: Net-(U2-Pad33) -> COL15
- U2 pad 36: Net-(U2-Pad36) -> COL14
- U2 pad 37: COL5 -> COL13
- U2 pad 4: COL14 -> ROW1
- U2 pad 40: Net-(U2-Pad40) -> COL12
- U2 pad 41: COL6 -> COL11
- U2 pad 42: COL7 -> COL10
- U2 pad 43: COL8 -> COL9
- U2 pad 44: COL9 -> COL16
- U2 pad 5: COL15 -> ROW2
- U2 pad 6: COL16 -> ROW3
- U2 pad 7: COL17 -> ROW4
Routing:
- net COL21: track 0.00 -> 361.5 mm, vias 0 -> 1
- net ROW5: track 518.7 -> 863.9 mm, vias 0 -> 2
- net ROW4: track 497.3 -> 832.4 mm, vias 0 -> 3
- net ROW3: track 465.1 -> 784.2 mm, vias 0 -> 6
- net COL20: track 0.00 -> 306.6 mm, vias 0 -> 2
- net COL15: track 409.3 -> 112.1 mm, vias 0 -> 1
- net ROW2: track 465.9 -> 754.3 mm, vias 2 -> 4
- net COL12: track 403.8 -> 155.6 mm
- net COL11: track 350.6 -> 112.0 mm
- net COL16: track 475.6 -> 247.1 mm, vias 3 -> 0
- net COL17: track 470.7 -> 253.8 mm, vias 2 -> 0
- net COL19: track 519.1 -> 320.0 mm, vias 2 -> 0
- net COL9: track 299.0 -> 106.8 mm, vias 3 -> 1
- net COL18: track 495.3 -> 303.8 mm, vias 2 -> 0
- net ROW1: track 506.0 -> 696.2 mm, vias 2 -> 4
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- added copper zone on B.Cu, net GND
- added copper zone on F.Cu, net GND
Other:
- board size 433.4 x 121.4 mm -> 433.4 x 126.2 mm
