File: 100plus/project/Rev2/100plus-2-secondusb.kicad_pcb (KiCad board)
At the start: 2 copper layers, 433.4 x 122.6 mm, 289 parts, among them J1 USB_Type_C_2.0_Receptacle, K1 KEYSW, K10 KEYSW, K100 KEYSW, K101 KEYSW, K102 KEYSW, K103 KEYSW, K104 KEYSW, K105 KEYSW, K106 KEYSW, K107 KEYSW, K108 KEYSW, K109 KEYSW, K11 KEYSW, K110 KEYSW, K111 KEYSW, K112 KEYSW, K113 KEYSW, K114 KEYSW, K115 KEYSW, K116 KEYSW, K117 KEYSW, K118 KEYSW, K119 KEYSW, K12 KEYSW, K120 KEYSW, K121 KEYSW, K122 KEYSW, K123 KEYSW, K124 KEYSW, K125 KEYSW, K126 KEYSW, K127 KEYSW, K128 KEYSW, K129 KEYSW, K13 KEYSW, K130 KEYSW, K14 KEYSW, K15 KEYSW, K16 KEYSW, K17 KEYSW, K18 KEYSW, K19 KEYSW, K2 KEYSW, K20 KEYSW, K21 KEYSW, K22 KEYSW, K23 KEYSW, K24 KEYSW, K25 KEYSW, K26 KEYSW, K27 KEYSW, K28 KEYSW, K29 KEYSW, K3 KEYSW, K30 KEYSW, K31 KEYSW, K32 KEYSW, K33 KEYSW, K34 KEYSW, K35 KEYSW, K36 KEYSW, K37 KEYSW, K38 KEYSW, K39 KEYSW, K4 KEYSW, K40 KEYSW, K41 KEYSW, K42 KEYSW, K43 KEYSW, K44 KEYSW, K45 KEYSW, K46 KEYSW, K47 KEYSW, K48 KEYSW, K49 KEYSW, K5 KEYSW, K50 KEYSW, K51 KEYSW, K52 KEYSW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

Commit message: nix 100plus 1 and 2 commits corrected usb
Parts:
- removed the J1 at (121.4, 73.8)
- added J1: USB_Type_C_2.0_Receptacle, Keyplus_conn_usb:USB_TypeC_U31F-24SNA0201, B.Cu at (121.4, 72.5)
- added J1: USB_Type_C_2.0_Receptacle, Keyplus_conn_usb:USB_TypeC_U31F-24SNA0201, B.Cu at (250.1, 72.4)
- added R1: 5.1k, Resistor_SMD:R_0603_1608Metric_Pad0.99x1.00mm_HandSolder, B.Cu at (127.1, 87.0)
- added R2: 5.1k, Resistor_SMD:R_0603_1608Metric_Pad0.99x1.00mm_HandSolder, B.Cu at (115.7, 86.9)
- moved R1 142.2 mm to (269.1, 83.3)
- moved R2 114.4 mm to (230.2, 86.6)
- moved REF** 58.5 mm to (319.1, 138.1)
Routing:
- net GND: track 248.2 -> 177.8 mm, vias 8 -> 9
- net Net-(J1-PadA5): track 15.3 -> 49.9 mm, vias 0 -> 2
- net Net-(J1-PadB5): track 12.4 -> 32.2 mm, vias 2 -> 4
- net Net-(J1-PadA6): track 163.5 -> 172.4 mm
- net +5V: track 270.3 -> 277.8 mm, vias 4 -> 7
- net Net-(J1-PadA7): track 159.2 -> 164.6 mm
- net COL4: track 195.6 -> 192.4 mm, vias 2 -> 1
- net ROW2: track 752.8 -> 754.3 mm
- net COL1: track 283.4 -> 284.8 mm
- net COL2: track 267.3 -> 268.7 mm
- net COL3: track 246.4 -> 247.7 mm
- net Net-(J1-PadA8): track 0.00 -> 0.53 mm
Other:
- board size 433.4 x 122.6 mm -> 433.4 x 123.8 mm
- net class VCC: trace_width 0.4 -> 0.5
