File: 100plus/project/Rev2/100plus-2.sch (KiCad schematic (older format))
At the start: 259 parts, among them J1 USB_Type_C_2.0_Receptacle, K1 KEYSW, K10 KEYSW, K100 KEYSW, K101 KEYSW, K102 KEYSW, K103 KEYSW, K104 KEYSW, K105 KEYSW, K106 KEYSW, K107 KEYSW, K108 KEYSW, K109 KEYSW, K11 KEYSW, K110 KEYSW, K111 KEYSW, K112 KEYSW, K113 KEYSW, K114 KEYSW, K115 KEYSW, K116 KEYSW, K117 KEYSW, K118 KEYSW, K119 KEYSW, K12 KEYSW, K120 KEYSW, K121 KEYSW, K122 KEYSW, K123 KEYSW, K124 KEYSW, K125 KEYSW, K126 KEYSW, K127 KEYSW, K128 KEYSW, K129 KEYSW, K13 KEYSW, K130 KEYSW, K14 KEYSW, K15 KEYSW, K16 KEYSW, K17 KEYSW, K18 KEYSW, K19 KEYSW, K2 KEYSW, K20 KEYSW, K21 KEYSW, K22 KEYSW, K23 KEYSW, K24 KEYSW, K25 KEYSW, K26 KEYSW, K27 KEYSW, K28 KEYSW, K29 KEYSW, K3 KEYSW, K30 KEYSW, K31 KEYSW, K32 KEYSW, K33 KEYSW, K34 KEYSW, K35 KEYSW, K36 KEYSW, K37 KEYSW, K38 KEYSW, K39 KEYSW, K4 KEYSW, K40 KEYSW, K41 KEYSW, K42 KEYSW, K43 KEYSW, K44 KEYSW, K45 KEYSW, K46 KEYSW, K47 KEYSW, K48 KEYSW, K49 KEYSW, K5 KEYSW, K50 KEYSW, K51 KEYSW, K52 KEYSW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

Commit message: 100 plus second revision
Parts:
- removed K129: KEYSW, Helpful:Kailh_MX_Socket, symbol keyboard_parts:KEYSW
- added K131, K132, K133, K135, K136: KEYSW, ai03_hybrid:MX-1.25U-NoLED, symbol keyboard_parts:KEYSW
- added K134: KEYSW, ai03_hybrid:MX-6.25U-NoLED, symbol keyboard_parts:KEYSW
Connections:
- wire segments 418 -> 429
Changed lines of the file:
@@
 	0    -1   -1   0
 $EndComp
-Wire Wire Line
-	15100 5400 15100 5350
 $Comp
 L keyboard_parts:KEYSW K82
@@
 $EndComp
 Wire Wire Line
-	4500 7400 4500 7300
+	4500 7400 4500 7350
 $Comp
 L keyboard_parts:KEYSW K114
@@
 $EndComp
 Wire Wire Line
-	6750 7400 6750 7300
-$Comp
-L keyboard_parts:KEYSW K110
-U 1 1 5B1A6898
-P 11500 7200
-F 0 "K110" H 11500 7433 60  0000 C CNN
-F 1 "KEYSW" H 11500 7100 60  0001 C CNN
-F 2 "Helpful:Kailh_MX_Socket" H 11500 7200 60  0001 C CNN
-F 3 "" H 11500 7200 60  0000 C CNN
-	1    11500 7200
-	1    0    0    -1
-$EndComp
+	6750 7400 6750 7350
 $Comp
 L Device:D D109
@@
 L keyboard_parts:KEYSW K116
 U 1 1 5B1A68A5
-P 11500 7300
-F 0 "K116" H 11500 7533 60  0000 C CNN
-F 1 "KEYSW" H 11500 7200 60  0001 C CNN
-F 2 "Helpful:Kailh_MX_Socket" H 11500 7300 60  0001 C CNN
-F 3 "" H 11500 7300 60  0000 C CNN
-	1    11500 7300
+P 11500 7250
+F 0 "K116" H 11500 7483 60  0000 C CNN
+F 1 "KEYSW" H 11500 7150 60  0001 C CNN
+F 2 "Helpful:Kailh_MX_Socket" H 11500 7250 60  0001 C CNN
+F 3 "" H 11500 7250 60  0000 C CNN
+	1    11500 7250
 	1    0    0    -1
 $EndComp
@@
 L keyboard_parts:KEYSW K126
 U 1 1 5B1A68B2
-P 11500 7400
-F 0 "K126" H 11500 7633 60  0000 C CNN
-F 1 "KEYSW" H 11500 7300 60  0001 C CNN
-F 2 "Helpful:Kailh_MX_Socket" H 11500 7400 60  0001 C CNN
-F 3 "" H 11500 7400 60  0000 C CNN
-	1    11500 7400
+P 11500 7350
+F 0 "K126" H 11500 7583 60  0000 C CNN
+F 1 "KEYSW" H 11500 7250 60  0001 C CNN
+F 2 "Helpful:Kailh_MX_Socket" H 11500 7350 60  0001 C CNN
+F 3 "" H 11500 7350 60  0000 C CNN
+	1    11500 7350
 	1    0    0    -1
 $EndComp
@@
 L keyboard_parts:KEYSW K127
 U 1 1 5B1A68CC
-P 12650 7400
-F 0 "K127" H 12650 7633 60  0000 C CNN
-F 1 "KEYSW" H 12650 7300 60  0001 C CNN
-F 2 "Helpful:Kailh_MX_Socket" H 12650 7400 60  0001 C CNN
-F 3 "" H 12650 7400 60  0000 C CNN
-	1    12650 7400
-	1    0    0    -1
-$EndComp
-$Comp
-L keyboard_parts:KEYSW K117
-U 1 1 5B1A68E6
 P 12650 7300
-F 0 "K117" H 12650 7533 60  0000 C CNN
+F 0 "K127" H 12650 7533 60  0000 C CNN
 F 1 "KEYSW" H 12650 7200 60  0001 C CNN
 F 2 "Helpful:Kailh_MX_Socket" H 12650 7300 60  0001 C CNN
 F 3 "" H 12650 7300 60  0000 C CNN
 	1    12650 7300
+	1    0    0    -1
+$EndComp
+$Comp
+L keyboard_parts:KEYSW K117
+U 1 1 5B1A68E6
+P 12650 7200
+F 0 "K117" H 12650 7433 60  0000 C CNN
+F 1 "KEYSW" H 12650 7100 60  0001 C CNN
+F 2 "Helpful:Kailh_MX_Socket" H 12650 7200 60  0001 C CNN
+F 3 "" H 12650 7200 60  0000 C CNN
+	1    12650 7200
 	1    0    0    -1
 $EndComp
@@
 $EndComp
 Wire Wire Line
-	13400 7400 13400 7300
+	13400 7400 13400 7350
 $Comp
 L keyboard_parts:KEYSW K119
@@
 Wire Wire Line
 	8750 7300 8750 7400
-Connection ~ 11200 7300
-Connection ~ 11200 7400
-Wire Wire Line
-	11200 7200 11200 7300
-Wire Wire Line
-	11200 7300 11200 7400
-Connection ~ 12350 7400
 Connection ~ 8750 7700
 Connection ~ 11200 7700
@@
 Connection ~ 12150 5300
 Wire Wire Line
-	11650 6300 11800 7200
-Connection ~ 11650 6300
-Wire Wire Line
-	11800 7200 11800 7300
-Connection ~ 11800 7200
-Connection ~ 11800 7300
-Wire Wire Line
-	11800 7300 11800 7400
-Wire Wire Line
 	12300 2400 12300 3350
 Connection ~ 12300 2400
@@
 	13750 5300 13250 6300
 Wire Wire Line
-	13250 6300 12950 7300
-Connection ~ 13250 6300
-Wire Wire Line
 	12950 7400 12950 7300
-Connection ~ 12950 7300
 Wire Wire Line
 	13500 2400 13900 3350
@@
 Text GLabel 25000 5250 2    50   Input ~ 0
 ROW5
-$Comp
-L keyboard_parts:KEYSW K129
-U 1 1 5B10B18E
-P 15400 5350
-F 0 "K129" H 15400 5583 60  0000 C CNN
-F 1 "KEYSW" H 15400 5250 60  0001 C CNN
-F 2 "Helpful:Kailh_MX_Socket" H 15400 5350 60  0001 C CNN
-F 3 "" H 15400 5350 60  0000 C CNN
-	1    15400 5350
-	-1   0    0    -1
-$EndComp
-Connection ~ 15100 5350
-Wire Wire Line
-	15100 5350 15100 5300
 Wire Wire Line
 	16500 4300 16500 4400
@@
 Wire Wire Line
 	15700 5350 15700 5300
-Connection ~ 15700 5350
 Connection ~ 15700 5300
 Text GLabel 23200 4050 0    50   Input ~ 0
@@
 $EndComp
 Wire Wire Line
-	5600 7400 5600 7300
+	5600 7400 5600 7350
 Connection ~ 5600 7700
 Wire Wire Line
@@
 Text GLabel 26050 3550 0    50   Input ~ 0
 COL21
+$Comp
+L keyboard_parts:KEYSW K131
+U 1 1 5B1C2F53
+P 4800 7350
+F 0 "K131" H 4800 7583 60  0000 C CNN
+F 1 "KEYSW" H 4800 7250 60  0001 C CNN
+F 2 "ai03_hybrid:MX-1.25U-NoLED" H 4800 7350 60  0001 C CNN
+F 3 "" H 4800 7350 60  0000 C CNN
+	1    4800 7350
+	1    0    0    -1
+$EndComp
+Connection ~ 4500 7350
+Wire Wire Line
+	4500 7350 4500 7300
+Wire Wire Line
+	5100 7350 5100 7300
+Connection ~ 5100 7300
+$Comp
+L keyboard_parts:KEYSW K132
+U 1 1 5B1E5103
+P 5900 7350
+F 0 "K132" H 5900 7583 60  0000 C CNN
+F 1 "KEYSW" H 5900 7250 60  0001 C CNN
+F 2 "ai03_hybrid:MX-1.25U-NoLED" H 5900 7350 60  0001 C CNN
+F 3 "" H 5900 7350 60  0000 C CNN
+	1    5900 7350
+	1    0    0    -1
+$EndComp
+Connection ~ 5600 7350
+Wire Wire Line
+	5600 7350 5600 7300
+Wire Wire Line
+	6200 7350 6200 7300
+Connection ~ 6200 7300
+$Comp
+L keyboard_parts:KEYSW K133
+U 1 1 5B207BC1
+P 7050 7350
+F 0 "K133" H 7050 7583 60  0000 C CNN
+F 1 "KEYSW" H 7050 7250 60  0001 C CNN
+F 2 "ai03_hybrid:MX-1.25U-NoLED" H 7050 7350 60  0001 C CNN
+F 3 "" H 7050 7350 60  0000 C CNN
+	1    7050 7350
+	1    0    0    -1
+$EndComp
+Connection ~ 6750 7350
+Wire Wire Line
+	6750 7350 6750 7300
+Wire Wire Line
+	7350 7350 7350 7300
+Connection ~ 7350 7300
+Connection ~ 11200 7250
+Connection ~ 11200 7350
+Wire Wire Line
+	11200 7350 11200 7400
+Connection ~ 11800 7250
+Connection ~ 11800 7350
+Wire Wire Line
+	11800 7350 11800 7400
+Wire Wire Line
+	11200 7250 11200 7350
+Wire Wire Line
+	11800 7250 11800 7350
+Wire Wire Line
+	11200 7150 11200 7250
+$Comp
+L keyboard_parts:KEYSW K110
+U 1 1 5B1A6898
+P 11500 7150
+F 0 "K110" H 11500 7383 60  0000 C CNN
+F 1 "KEYSW" H 11500 7050 60  0001 C CNN
+F 2 "Helpful:Kailh_MX_Socket" H 11500 7150 60  0001 C CNN
+F 3 "" H 11500 7150 60  0000 C CNN
+	1    11500 7150
+	1    0    0    -1
+$EndComp
+Wire Wire Line
+	11800 7150 11800 7250
+$Comp
+L keyboard_parts:KEYSW K135
+U 1 1 5B2BC4CD
+P 11500 7400
+F 0 "K135" H 11500 7633 60  0000 C CNN
+F 1 "KEYSW" H 11500 7300 60  0001 C CNN
+F 2 "ai03_hybrid:MX-1.25U-NoLED" H 11500 7400 60  0001 C CNN
+F 3 "" H 11500 7400 60  0000 C CNN
+	1    11500 7400
+	1    0    0    -1
+$EndComp
+Connection ~ 11200 7400
+Wire Wire Line
+	11650 6300 11800 7150
+Connection ~ 11650 6300
+Connection ~ 11800 7150
+$Comp
+L keyboard_parts:KEYSW K136
+U 1 1 5B3287A8
+P 12650 7400
+F 0 "K136" H 12650 7633 60  0000 C CNN
+F 1 "KEYSW" H 12650 7300 60  0001 C CNN
+F 2 "ai03_hybrid:MX-1.25U-NoLED" H 12650 7400 60  0001 C CNN
+F 3 "" H 12650 7400 60  0000 C CNN
+	1    12650 7400
+	1    0    0    -1
+$EndComp
+Connection ~ 12350 7400
+Wire Wire Line
+	12950 7300 12950 7200
+Connection ~ 12950 7300
+Wire Wire Line
+	12350 7300 12350 7200
+Connection ~ 12350 7300
+Wire Wire Line
+	12950 7200 13250 6300
+Connection ~ 12950 7200
+Connection ~ 13250 6300
+$Comp
+L keyboard_parts:KEYSW K134
+U 1 1 5B3DD4AB
+P 13700 7350
+F 0 "K134" H 13700 7583 60  0000 C CNN
+F 1 "KEYSW" H 13700 7250 60  0001 C CNN
+F 2 "ai03_hybrid:MX-6.25U-NoLED" H 13700 7350 60  0001 C CNN
+F 3 "" H 13700 7350 60  0000 C CNN
+	1    13700 7350
+	1    0    0    -1
+$EndComp
+Connection ~ 13400 7350
+Wire Wire Line
+	13400 7350 13400 7300
+Wire Wire Line
+	14000 7350 14000 7300
+Connection ~ 14000 7300
+Wire Wire Line
+	15100 5300 15100 5400
 $EndSCHEMATC
