File: 100plus/project/Rev2/100plus-2.kicad_pcb (KiCad board)
At the start: 2 copper layers, 433.4 x 122.6 mm, 289 parts, among them J1 USB_Type_C_2.0_Receptacle, K1 KEYSW, K10 KEYSW, K100 KEYSW, K101 KEYSW, K102 KEYSW, K103 KEYSW, K104 KEYSW, K105 KEYSW, K106 KEYSW, K107 KEYSW, K108 KEYSW, K109 KEYSW, K11 KEYSW, K110 KEYSW, K111 KEYSW, K112 KEYSW, K113 KEYSW, K114 KEYSW, K115 KEYSW, K116 KEYSW, K117 KEYSW, K118 KEYSW, K119 KEYSW, K12 KEYSW, K120 KEYSW, K121 KEYSW, K122 KEYSW, K123 KEYSW, K124 KEYSW, K125 KEYSW, K126 KEYSW, K127 KEYSW, K128 KEYSW, K129 KEYSW, K13 KEYSW, K130 KEYSW, K14 KEYSW, K15 KEYSW, K16 KEYSW, K17 KEYSW, K18 KEYSW, K19 KEYSW, K2 KEYSW, K20 KEYSW, K21 KEYSW, K22 KEYSW, K23 KEYSW, K24 KEYSW, K25 KEYSW, K26 KEYSW, K27 KEYSW, K28 KEYSW, K29 KEYSW, K3 KEYSW, K30 KEYSW, K31 KEYSW, K32 KEYSW, K33 KEYSW, K34 KEYSW, K35 KEYSW, K36 KEYSW, K37 KEYSW, K38 KEYSW, K39 KEYSW, K4 KEYSW, K40 KEYSW, K41 KEYSW, K42 KEYSW, K43 KEYSW, K44 KEYSW, K45 KEYSW, K46 KEYSW, K47 KEYSW, K48 KEYSW, K49 KEYSW, K5 KEYSW, K50 KEYSW, K51 KEYSW, K52 KEYSW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

Commit message: 100 plus second revision
Parts:
- removed K129: KEYSW, ai03_hybrid:MX-2U-NoLED
- added K131: KEYSW, ai03_hybrid:MX-1.25U-NoLED, F.Cu at (109.5, 185.7)
- added K132: KEYSW, ai03_hybrid:MX-1.25U-NoLED, F.Cu at (133.4, 185.7)
- added K133: KEYSW, ai03_hybrid:MX-1.25U-NoLED, F.Cu at (157.2, 185.7)
- added K134: KEYSW, ai03_hybrid:MX-6.25U-NoLED, F.Cu at (228.6, 185.7)
- added K135: KEYSW, ai03_hybrid:MX-1.25U-NoLED, F.Cu at (300.0, 185.7)
- added K136: KEYSW, ai03_hybrid:MX-1.25U-NoLED, F.Cu at (323.9, 185.7)
Routing:
- net Net-(D110-Pad2): track 27.5 -> 53.5 mm
- net Net-(D111-Pad2): track 28.6 -> 45.1 mm
- net COL10: track 130.9 -> 143.6 mm
- net GND: track 248.2 -> 260.8 mm, vias 8 -> 9
- net COL14: track 215.3 -> 203.4 mm
- net Net-(D112-Pad2): track 9.54 -> 20.1 mm
- net Net-(D108-Pad2): track 10.1 -> 19.1 mm
- net Net-(D120-Pad2): track 9.44 -> 18.3 mm
- net Net-(D107-Pad2): track 9.35 -> 17.4 mm
- net COL2: track 267.3 -> 274.4 mm
- net COL13: track 176.3 -> 182.3 mm
- net ROW2: track 752.8 -> 747.2 mm
- net COL12: track 155.6 -> 160.8 mm
- net COL5: track 197.0 -> 200.2 mm
- net Net-(D78-Pad2): track 12.0 -> 9.44 mm
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
Commit message: 100 plus second revision
Other:
- board text added: "PCB by amesa0 (Helpful) - Revision 2"
- board text removed: "PCB by amesa0 (Helpful) - Revision 1"
Changed lines of the file:
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@@
   (gr_line (start 485.775 80.9625) (end 485.775 195.2625) (layer Edge.Cuts) (width 0.2))
   (gr_line (start 259.55625 78.58125) (end 483.39375 78.58125) (layer Edge.Cuts) (width 0.2))
-  (gr_text "PCB by amesa0 (Helpful) - Revision 1" (at 163.75 114.9) (layer F.SilkS)
+  (gr_text "PCB by amesa0 (Helpful) - Revision 2" (at 163.75 114.9) (layer F.SilkS)
     (effects (font (size 3 3) (thickness 0.6)))
   )
