File: 100plus/project/Rev2/100plus-2.kicad_pcb (KiCad board)
At the start: 2 copper layers, 433.4 x 122.6 mm, 294 parts, among them J1 USB_Type_C_2.0_Receptacle, K1 KEYSW, K10 KEYSW, K100 KEYSW, K101 KEYSW, K102 KEYSW, K103 KEYSW, K104 KEYSW, K105 KEYSW, K106 KEYSW, K107 KEYSW, K108 KEYSW, K109 KEYSW, K11 KEYSW, K110 KEYSW, K111 KEYSW, K112 KEYSW, K113 KEYSW, K114 KEYSW, K115 KEYSW, K116 KEYSW, K117 KEYSW, K118 KEYSW, K119 KEYSW, K12 KEYSW, K120 KEYSW, K121 KEYSW, K122 KEYSW, K123 KEYSW, K124 KEYSW, K125 KEYSW, K126 KEYSW, K127 KEYSW, K128 KEYSW, K13 KEYSW, K130 KEYSW, K131 KEYSW, K132 KEYSW, K133 KEYSW, K134 KEYSW, K135 KEYSW, K136 KEYSW, K14 KEYSW, K15 KEYSW, K16 KEYSW, K17 KEYSW, K18 KEYSW, K19 KEYSW, K2 KEYSW, K20 KEYSW, K21 KEYSW, K22 KEYSW, K23 KEYSW, K24 KEYSW, K25 KEYSW, K26 KEYSW, K27 KEYSW, K28 KEYSW, K29 KEYSW, K3 KEYSW, K30 KEYSW, K31 KEYSW, K32 KEYSW, K33 KEYSW, K34 KEYSW, K35 KEYSW, K36 KEYSW, K37 KEYSW, K38 KEYSW, K39 KEYSW, K4 KEYSW, K40 KEYSW, K41 KEYSW, K42 KEYSW, K43 KEYSW, K44 KEYSW, K45 KEYSW, K46 KEYSW, K47 KEYSW, K48 KEYSW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

Commit message: 100plus layout changes
Routing:
- net ROW0: track 669.9 -> 658.3 mm
- net ROW2: track 753.7 -> 747.2 mm
- net ROW1: track 700.7 -> 696.1 mm
- net GND: track 261.4 -> 260.8 mm
- net COL19: track 321.3 -> 320.8 mm
Other:
- board text added: "Design guidance from Amtra5, _spindle, woodkeys, Hiney, ai03"
- board text removed: "Design guidance from Amtra5, _spindle, woodkeys, hiney, ai03"
