File: 100plus/project/Rev2/Project/100plus-2.sch (KiCad schematic (older format))
At the start: 264 parts, among them J1 USB_Type_C_2.0_Receptacle, K1 KEYSW, K10 KEYSW, K100 KEYSW, K101 KEYSW, K102 KEYSW, K103 KEYSW, K104 KEYSW, K105 KEYSW, K106 KEYSW, K107 KEYSW, K108 KEYSW, K109 KEYSW, K11 KEYSW, K110 KEYSW, K111 KEYSW, K112 KEYSW, K113 KEYSW, K114 KEYSW, K115 KEYSW, K116 KEYSW, K117 KEYSW, K118 KEYSW, K119 KEYSW, K12 KEYSW, K120 KEYSW, K121 KEYSW, K122 KEYSW, K123 KEYSW, K124 KEYSW, K125 KEYSW, K126 KEYSW, K127 KEYSW, K128 KEYSW, K13 KEYSW, K130 KEYSW, K131 KEYSW, K132 KEYSW, K133 KEYSW, K134 KEYSW, K135 KEYSW, K136 KEYSW, K14 KEYSW, K15 KEYSW, K16 KEYSW, K17 KEYSW, K18 KEYSW, K19 KEYSW, K2 KEYSW, K20 KEYSW, K21 KEYSW, K22 KEYSW, K23 KEYSW, K24 KEYSW, K25 KEYSW, K26 KEYSW, K27 KEYSW, K28 KEYSW, K29 KEYSW, K3 KEYSW, K30 KEYSW, K31 KEYSW, K32 KEYSW, K33 KEYSW, K34 KEYSW, K35 KEYSW, K36 KEYSW, K37 KEYSW, K38 KEYSW, K39 KEYSW, K4 KEYSW, K40 KEYSW, K41 KEYSW, K42 KEYSW, K43 KEYSW, K44 KEYSW, K45 KEYSW, K46 KEYSW, K47 KEYSW, K48 KEYSW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

Commit message: 100plus layout changes
Parts:
- removed K43: KEYSW, Helpful:Kailh_MX_Socket, symbol keyboard_parts:KEYSW
Connections:
- wire segments 429 -> 428
Changed lines of the file:
@@
-$EndComp
-$Comp
-L keyboard_parts:KEYSW K43
-U 1 1 5B0CF8D8
-P 15200 3450
-F 0 "K43" H 15200 3683 60  0000 C CNN
-F 1 "KEYSW" H 15200 3350 60  0001 C CNN
-F 2 "Helpful:Kailh_MX_Socket" H 15200 3450 60  0001 C CNN
-F 3 "" H 15200 3450 60  0000 C CNN
-	1    15200 3450
-	1    0    0    -1
 $EndComp
 $Comp
@@
 	15100 2400 15500 3350
 Connection ~ 15100 2400
-Connection ~ 14900 3450
-Wire Wire Line
-	15500 3350 15500 3450
-Connection ~ 15500 3350
 Wire Wire Line
 	15900 2400 16300 3350
