File: 100plus/project/Rev3/Project_current/_autosave-100plus-2.kicad_pcb (KiCad board)
At the start: 2 copper layers, 433.4 x 123.8 mm, 320 parts, among them J1 USB_Type_C_2.0_Receptacle, K1 KEYSW, K10 KEYSW, K100 KEYSW, K101 KEYSW, K102 KEYSW, K103 KEYSW, K104 KEYSW, K105 KEYSW, K106 KEYSW, K107 KEYSW, K108 KEYSW, K109 KEYSW, K11 KEYSW, K110 KEYSW, K111 KEYSW, K112 KEYSW, K113 KEYSW, K114 KEYSW, K115 KEYSW, K116 KEYSW, K117 KEYSW, K118 KEYSW, K119 KEYSW, K12 KEYSW, K120 KEYSW, K121 KEYSW, K122 KEYSW, K123 KEYSW, K124 KEYSW, K125 KEYSW, K126 KEYSW, K127 KEYSW, K128 KEYSW, K129 KEYSW, K13 KEYSW, K130 KEYSW, K131 KEYSW, K132 KEYSW, K133 KEYSW, K134 KEYSW, K135 KEYSW, K136 KEYSW, K137 KEYSW, K138 KEYSW, K139 KEYSW, K14 KEYSW, K143 KEYSW, K144 KEYSW, K145 KEYSW, K146 KEYSW, K147 KEYSW, K148 KEYSW, K149 KEYSW, K15 KEYSW, K150 KEYSW, K151 KEYSW, K152 KEYSW, K153 KEYSW, K154 KEYSW, K155 KEYSW, K156 KEYSW, K157 KEYSW, K158 KEYSW, K159 KEYSW, K16 KEYSW, K160 KEYSW, K165 KEYSW, K166 KEYSW, K167 KEYSW, K168 KEYSW, K169 KEYSW, K17 KEYSW, K170 KEYSW, K171 KEYSW, K172 KEYSW, K173 KEYSW, K174 KEYSW, K175 KEYSW, K176 KEYSW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

Commit message: mostly 100plus corrections
Parts:
- removed K49: KEYSW, ai03_hybrid:MX-1U-NoLED
Changed lines of the file:
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@@
     (tracks 1103)
     (zones 0)
-    (modules 320)
+    (modules 319)
     (nets 235)
   )
@@
   )
   (module ai03_hybrid:MX-1U-NoLED (layer F.Cu)
-    (at 154.78125 128.5875)
-    (fp_text reference K49 (at 0 3.175) (layer Dwgs.User)
-      (effects (font (size 1 1) (thickness 0.15)))
-    )
-    (fp_text value KEYSW (at 0 -7.9375) (layer Dwgs.User)
-      (effects (font (size 1 1) (thickness 0.15)))
-    )
-    (fp_line (start -9.525 9.525) (end -9.525 -9.525) (layer Dwgs.User) (width 0.15))
-    (fp_line (start 9.525 9.525) (end -9.525 9.525) (layer Dwgs.User) (width 0.15))
-    (fp_line (start 9.525 -9.525) (end 9.525 9.525) (layer Dwgs.User) (width 0.15))
-    (fp_line (start -9.525 -9.525) (end 9.525 -9.525) (layer Dwgs.User) (width 0.15))
-    (fp_line (start -7 -7) (end -7 -5) (layer Dwgs.User) (width 0.15))
-    (fp_line (start -5 -7) (end -7 -7) (layer Dwgs.User) (width 0.15))
-    (fp_line (start -7 7) (end -5 7) (layer Dwgs.User) (width 0.15))
-    (fp_line (start -7 5) (end -7 7) (layer Dwgs.User) (width 0.15))
-    (fp_line (start 7 7) (end 7 5) (layer Dwgs.User) (width 0.15))
-    (fp_line (start 5 7) (end 7 7) (layer Dwgs.User) (width 0.15))
-    (fp_line (start 7 -7) (end 7 -5) (layer Dwgs.User) (width 0.15))
-    (fp_line (start 5 -7) (end 7 -7) (layer Dwgs.User) (width 0.15))
-    (pad "" np_thru_hole circle (at 5.08 0 48.0996) (size 1.75 1.75) (drill 1.75) (layers *.Cu *.Mask))
-    (pad "" np_thru_hole circle (at -5.08 0 48.0996) (size 1.75 1.75) (drill 1.75) (layers *.Cu *.Mask))
-    (pad 1 thru_hole circle (at -2.5 -4) (size 2.25 2.25) (drill 1.47) (layers *.Cu B.Mask)
-      (net 138 COL4))
-    (pad "" np_thru_hole circle (at 0 0) (size 3.9878 3.9878) (drill 3.9878) (layers *.Cu *.Mask))
-    (pad 1 thru_hole oval (at -3.81 -2.54 48.0996) (size 4.211556 2.25) (drill 1.47 (offset 0.980778 0)) (layers *.Cu B.Mask)
-      (net 138 COL4))
-    (pad 2 thru_hole circle (at 2.54 -5.08) (size 2.25 2.25) (drill 1.47) (layers *.Cu B.Mask)
-      (net 50 "Net-(D47-Pad2)"))
-    (pad 2 thru_hole oval (at 2.5 -4.5 86.0548) (size 2.831378 2.25) (drill 1.47 (offset 0.290689 0)) (layers *.Cu B.Mask)
-      (net 50 "Net-(D47-Pad2)"))
-  )
-  (module ai03_hybrid:MX-1U-NoLED (layer F.Cu)
