File: 100plus/project/Rev3/Project_current/_saved_100plus-2.sch (KiCad schematic (older format))
At the start: 314 parts, among them J1 USB_Type_C_2.0_Receptacle, K1 KEYSW, K10 KEYSW, K100 KEYSW, K101 KEYSW, K102 KEYSW, K103 KEYSW, K104 KEYSW, K105 KEYSW, K106 KEYSW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

Commit message: mostly 100plus corrections
Parts:
- added U3, U?: Teensy2.0++, keebs_misc:Teensy2.0++, symbol keyboard_parts:Teensy2.0++
Connections:
- wire segments 526 -> 524
