File: 100plus/project/Rev3/Project_current/100plus-2.kicad_pcb (KiCad board)
At the start: 2 copper layers, 433.4 x 123.8 mm, 320 parts, among them J1 USB_Type_C_2.0_Receptacle, K1 KEYSW, K10 KEYSW, K100 KEYSW, K101 KEYSW, K102 KEYSW, K103 KEYSW, K104 KEYSW, K105 KEYSW, K106 KEYSW, K107 KEYSW, K108 KEYSW, K109 KEYSW, K11 KEYSW, K110 KEYSW, K111 KEYSW, K112 KEYSW, K113 KEYSW, K114 KEYSW, K115 KEYSW, K116 KEYSW, K117 KEYSW, K118 KEYSW, K119 KEYSW, K12 KEYSW, K120 KEYSW, K121 KEYSW, K122 KEYSW, K123 KEYSW, K124 KEYSW, K125 KEYSW, K126 KEYSW, K127 KEYSW, K128 KEYSW, K129 KEYSW, K13 KEYSW, K130 KEYSW, K131 KEYSW, K132 KEYSW, K133 KEYSW, K134 KEYSW, K135 KEYSW, K136 KEYSW, K137 KEYSW, K138 KEYSW, K139 KEYSW, K14 KEYSW, K143 KEYSW, K144 KEYSW, K145 KEYSW, K146 KEYSW, K147 KEYSW, K148 KEYSW, K149 KEYSW, K15 KEYSW, K150 KEYSW, K151 KEYSW, K152 KEYSW, K153 KEYSW, K154 KEYSW, K155 KEYSW, K156 KEYSW, K157 KEYSW, K158 KEYSW, K159 KEYSW, K16 KEYSW, K160 KEYSW, K165 KEYSW, K166 KEYSW, K167 KEYSW, K168 KEYSW, K169 KEYSW, K17 KEYSW, K170 KEYSW, K171 KEYSW, K172 KEYSW, K173 KEYSW, K174 KEYSW, K175 KEYSW, K176 KEYSW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

Commit message: fake alice
Parts:
- removed the U3 at (-17.5, 91.8)
- removed the U3 at (-19.6, 117.2)
- removed the U3 at (392.9, 100.0)
- removed the U3 at (107.2, 100.0)
- added B2: SPARKFUN_PRO_MICRO, Boards:SPARKFUN_PRO_MICRO, B.Cu at (469.4, 108.2)
- added U3: Teensy2.0++, keebs_misc:Teensy2.0++, B.Cu at (392.7, 103.1)
- added U6: Teensy2.0++, keebs_misc:Teensy2.0++, B.Cu at (392.4, 126.0)
- moved U2 200.3 mm to (-46.0, 37.8)
- moved B1 66.5 mm to (435.8, 90.4)
- moved D18 7.92 mm to (435.2, 101.2), turned to 0 degrees
- moved D16 7.15 mm to (392.3, 100.8), turned to 0 degrees
- moved D41 6.11 mm to (461.5, 121.2)
- moved D42 5.54 mm to (480.4, 120.5)
- moved D37 2.75 mm to (380.4, 121.4)
- moved D20 1.52 mm to (481.1, 104.6)
- moved D19 1.52 mm to (462.0, 104.6)
Routing:
- net Net-(D41-Pad2): track 9.69 -> 18.0 mm
- net Net-(D42-Pad2): track 9.67 -> 17.6 mm
- net ROW1: track 428.4 -> 424.4 mm, vias 2 -> 0
- net Net-(D16-Pad2): track 24.1 -> 21.7 mm
- net Net-(D19-Pad2): track 21.6 -> 24.0 mm
- net Net-(D37-Pad2): track 28.8 -> 27.1 mm
- net Net-(D20-Pad2): track 22.2 -> 23.8 mm
- net Net-(D18-Pad2): track 21.6 -> 20.4 mm
- net ROW0: track 460.6 -> 459.7 mm
- net Net-(D35-Pad2): track 11.3 -> 11.2 mm, vias 1 -> 0
