File: 100plus/project/Rev3/Project_current/100plus-2.sch (KiCad schematic (older format))
At the start: 314 parts, among them J1 USB_Type_C_2.0_Receptacle, K1 KEYSW, K10 KEYSW, K100 KEYSW, K101 KEYSW, K102 KEYSW, K103 KEYSW, K104 KEYSW, K105 KEYSW, K106 KEYSW, K107 KEYSW, K108 KEYSW, K109 KEYSW, K11 KEYSW, K110 KEYSW, K111 KEYSW, K112 KEYSW, K113 KEYSW, K114 KEYSW, K115 KEYSW, K116 KEYSW, K117 KEYSW, K118 KEYSW, K119 KEYSW, K12 KEYSW, K120 KEYSW, K121 KEYSW, K122 KEYSW, K123 KEYSW, K124 KEYSW, K125 KEYSW, K126 KEYSW, K127 KEYSW, K128 KEYSW, K129 KEYSW, K13 KEYSW, K130 KEYSW, K131 KEYSW, K132 KEYSW, K133 KEYSW, K134 KEYSW, K135 KEYSW, K136 KEYSW, K137 KEYSW, K138 KEYSW, K139 KEYSW, K14 KEYSW, K143 KEYSW, K144 KEYSW, K145 KEYSW, K146 KEYSW, K147 KEYSW, K148 KEYSW, K149 KEYSW, K15 KEYSW, K150 KEYSW, K152 KEYSW, K153 KEYSW, K154 KEYSW, K155 KEYSW, K156 KEYSW, K157 KEYSW, K158 KEYSW, K159 KEYSW, K16 KEYSW, K160 KEYSW, K165 KEYSW, K166 KEYSW, K167 KEYSW, K168 KEYSW, K169 KEYSW, K17 KEYSW, K170 KEYSW, K171 KEYSW, K172 KEYSW, K173 KEYSW, K174 KEYSW, K175 KEYSW, K176 KEYSW, K177 KEYSW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

Commit message: mostly 100plus corrections
Parts:
- added U3: Teensy2.0++, keebs_misc:Teensy2.0++, symbol keyboard_parts:Teensy2.0++
Connections:
- wire segments 526 -> 524
Changed lines of the file:
@@
 Connection ~ 10250 7150
 Connection ~ 10250 7300
-Wire Wire Line
-	10250 7300 10250 7350
 $Comp
 L keyboard_parts:KEYSW K169
@@
 Connection ~ 14000 7250
 Wire Wire Line
-	10250 7400 10250 7350
-Connection ~ 10250 7350
-Wire Wire Line
-	10250 7350 10250 7300
-Wire Wire Line
 	10250 7150 10250 7300
 Wire Wire Line
 	9650 7150 9650 7300
+$Comp
+L keyboard_parts:Teensy2.0++ U3
+U 1 1 5B40C5BD
+P 26650 6650
+F 0 "U3" H 26650 8297 60  0000 C CNN
+F 1 "Teensy2.0++" H 26650 8191 60  0000 C CNN
+F 2 "keebs_misc:Teensy2.0++" H 26650 6700 60  0001 C CNN
+F 3 "" H 26650 6700 60  0000 C CNN
+	1    26650 6650
+	1    0    0    -1
+$EndComp
+Text GLabel 28200 6650 2    50   Input ~ 0
+ROW0
+Text GLabel 28200 6100 2    50   Input ~ 0
+ROW1
+Text GLabel 28200 6200 2    50   Input ~ 0
+ROW2
+Text GLabel 28200 6300 2    50   Input ~ 0
+ROW3
+Text GLabel 28200 6400 2    50   Input ~ 0
+ROW4
+Text GLabel 28200 6550 2    50   Input ~ 0
+ROW5
+Text GLabel 28200 5950 2    50   Input ~ 0
+COL19
+Text GLabel 28200 5850 2    50   Input ~ 0
+COL18
+Text GLabel 28200 5750 2    50   Input ~ 0
+COL17
+Text GLabel 28200 5650 2    50   Input ~ 0
+COL16
+Text GLabel 28200 5250 2    50   Input ~ 0
+COL12
+Text GLabel 28200 5350 2    50   Input ~ 0
+COL11
+Text GLabel 28200 5450 2    50   Input ~ 0
+COL10
+Text GLabel 28200 5550 2    50   Input ~ 0
+COL9
+Text GLabel 28200 7050 2    50   Input ~ 0
+COL8
+Text GLabel 28200 6950 2    50   Input ~ 0
+COL7
+Text GLabel 28200 6850 2    50   Input ~ 0
+COL6
+Text GLabel 28200 7150 2    50   Input ~ 0
+COL4
+Text GLabel 28200 7250 2    50   Input ~ 0
+COL3
+Text GLabel 28200 6750 2    50   Input ~ 0
+COL5
+Wire Wire Line
+	10250 7300 10250 7400
+Text GLabel 29250 6500 0    50   Input ~ 0
+COL0
+Text GLabel 29250 6400 0    50   Input ~ 0
+COL1
+Text GLabel 29250 6300 0    50   Input ~ 0
+COL2
+Text GLabel 29250 6150 0    50   Input ~ 0
+COL15
+Text GLabel 29250 5600 0    50   Input ~ 0
+COL14
+Text GLabel 29250 6050 0    50   Input ~ 0
+COL20
+Text GLabel 29250 6800 0    50   Input ~ 0
+COL21
+Text GLabel 29250 5700 0    50   Input ~ 0
+COL13
 $EndSCHEMATC

Commit message: fake alice
Parts:
- added B2: SPARKFUN_PRO_MICRO, Boards:SPARKFUN_PRO_MICRO, symbol SparkFun-Boards:SPARKFUN_PRO_MICRO
- added U6: Teensy2.0++, keebs_misc:Teensy2.0++, symbol keyboard_parts:Teensy2.0++
Changed lines of the file:
@@
 Text GLabel 29250 5700 0    50   Input ~ 0
 COL13
+$Comp
+L keyboard_parts:Teensy2.0++ U6
+U 1 1 5B465502
+P 20450 10000
+F 0 "U6" H 20450 11647 60  0000 C CNN
+F 1 "Teensy2.0++" H 20450 11541 60  0000 C CNN
+F 2 "keebs_misc:Teensy2.0++" H 20450 10050 60  0001 C CNN
+F 3 "" H 20450 10050 60  0000 C CNN
+	1    20450 10000
+	1    0    0    -1
+$EndComp
+$Comp
+L SparkFun-Boards:SPARKFUN_PRO_MICRO B2
+U 1 1 5B486C68
+P 28600 3750
+F 0 "B2" H 28600 4660 45  0000 C CNN
+F 1 "SPARKFUN_PRO_MICRO" H 28600 4576 45  0000 C CNN
+F 2 "Boards:SPARKFUN_PRO_MICRO" H 28600 4550 20  0001 C CNN
+F 3 "" H 28600 3750 50  0001 C CNN
+F 4 "XXX-00000" H 28600 4481 60  0000 C CNN "Field4"
+	1    28600 3750
+	1    0    0    -1
+$EndComp
+Text GLabel 29050 4200 2    50   Input ~ 0
+COL18
+Text GLabel 29050 4300 2    50   Input ~ 0
+COL19
+Text GLabel 28150 3800 0    50   Input ~ 0
+ROW0
+Text GLabel 28150 4300 0    50   Input ~ 0
+ROW1
+Text GLabel 28150 4100 0    50   Input ~ 0
+ROW3
+Text GLabel 28150 4200 0    50   Input ~ 0
+ROW2
+Text GLabel 28150 4000 0    50   Input ~ 0
+ROW4
+Text GLabel 28150 3900 0    50   Input ~ 0
+ROW5
+Text GLabel 28150 3600 0    50   Input ~ 0
+COL20
+Text GLabel 28150 3700 0    50   Input ~ 0
+COL21
 $EndSCHEMATC
