File: alice/alice/alice.kicad_pcb (KiCad board)
At the start: 2 copper layers, 358.6 x 135.4 mm, 160 parts, among them J1 USB_mini_micro_B, K1 KEYSW, K10 KEYSW, K11 KEYSW, K12 KEYSW, K13 KEYSW, K14 KEYSW, K15 KEYSW, K16 KEYSW, K17 KEYSW, K18 KEYSW, K19 KEYSW, K2 KEYSW, K20 KEYSW, K21 KEYSW, K22 KEYSW, K23 KEYSW, K24 KEYSW, K25 KEYSW, K26 KEYSW, K27 KEYSW, K28 KEYSW, K29 KEYSW, K3 KEYSW, K30 KEYSW, K31 KEYSW, K32 KEYSW, K33 KEYSW, K34 KEYSW, K35 KEYSW, K36 KEYSW, K37 KEYSW, K38 KEYSW, K39 KEYSW, K4 KEYSW, K40 KEYSW, K41 KEYSW, K42 KEYSW, K43 KEYSW, K44 KEYSW, K45 KEYSW, K46 KEYSW, K47 KEYSW, K48 KEYSW, K49 KEYSW, K5 KEYSW, K50 KEYSW, K51 KEYSW, K52 KEYSW, K53 KEYSW, K54 KEYSW, K55 KEYSW, K56 KEYSW, K57 KEYSW, K58 KEYSW, K59 KEYSW, K6 KEYSW, K60 KEYSW, K61 KEYSW, K62 KEYSW, K63 KEYSW, K64 KEYSW, K65 KEYSW, K66 KEYSW, K67 KEYSW, K68 KEYSW, K69 KEYSW, K7 KEYSW, K70 KEYSW, K71 KEYSW, K72 KEYSW, K73 KEYSW, K74 KEYSW, K8 KEYSW, K9 KEYSW, SW1 SW_PUSH, U1 ATMEGA32U4, Y1 Crystal_GND24

Commit message: falice
Parts:
- moved K65 0.18 mm to (279.1, 213.1)
- moved K64 0.18 mm to (248.8, 206.7)
- moved K68 0.09 mm to (213.2, 202.5)
Connections:
- D1 pad 1: Net-(D1-Pad1) -> row0
- D10 pad 1: Net-(D1-Pad1) -> row0
- D11 pad 1: Net-(D1-Pad1) -> row0
- D12 pad 1: Net-(D1-Pad1) -> row0
- D13 pad 1: Net-(D1-Pad1) -> row0
- D14 pad 1: Net-(D1-Pad1) -> row0
- D15 pad 1: Net-(D1-Pad1) -> row0
- D16 pad 1: Net-(D1-Pad1) -> row0
- D17 pad 1: Net-(D17-Pad1) -> row1
- D18 pad 1: Net-(D17-Pad1) -> row1
- D19 pad 1: Net-(D17-Pad1) -> row1
- D2 pad 1: Net-(D1-Pad1) -> row0
- D20 pad 1: Net-(D17-Pad1) -> row1
- D21 pad 1: Net-(D17-Pad1) -> row1
- D22 pad 1: Net-(D17-Pad1) -> row1
- D23 pad 1: Net-(D17-Pad1) -> row1
- D24 pad 1: Net-(D17-Pad1) -> row1
- D25 pad 1: Net-(D17-Pad1) -> row1
- D26 pad 1: Net-(D17-Pad1) -> row1
- D27 pad 1: Net-(D17-Pad1) -> row1
- D28 pad 1: Net-(D17-Pad1) -> row1
- D29 pad 1: Net-(D17-Pad1) -> row1
- D3 pad 1: Net-(D1-Pad1) -> row0
- D30 pad 1: Net-(D17-Pad1) -> row1
- D31 pad 1: Net-(D17-Pad1) -> row1
- D32 pad 1: Net-(D32-Pad1) -> row2
- D33 pad 1: Net-(D32-Pad1) -> row2
- D34 pad 1: Net-(D32-Pad1) -> row2
- D35 pad 1: Net-(D32-Pad1) -> row2
- D36 pad 1: Net-(D32-Pad1) -> row2
- D37 pad 1: Net-(D32-Pad1) -> row2
- D38 pad 1: Net-(D32-Pad1) -> row2
- D39 pad 1: Net-(D32-Pad1) -> row2
- D4 pad 1: Net-(D1-Pad1) -> row0
- D40 pad 1: Net-(D32-Pad1) -> row2
- D41 pad 1: Net-(D32-Pad1) -> row2
- D42 pad 1: Net-(D32-Pad1) -> row2
- D43 pad 1: Net-(D32-Pad1) -> row2
- D44 pad 1: Net-(D32-Pad1) -> row2
- D45 pad 1: Net-(D32-Pad1) -> row2
- D46 pad 1: Net-(D46-Pad1) -> row3
- D47 pad 1: Net-(D46-Pad1) -> row3
- D48 pad 1: Net-(D46-Pad1) -> row3
- D49 pad 1: Net-(D46-Pad1) -> row3
- D5 pad 1: Net-(D1-Pad1) -> row0
- D50 pad 1: Net-(D46-Pad1) -> row3
- D51 pad 1: Net-(D46-Pad1) -> row3
- D52 pad 1: Net-(D46-Pad1) -> row3
- D53 pad 1: Net-(D46-Pad1) -> row3
- D54 pad 1: Net-(D46-Pad1) -> row3
- D55 pad 1: Net-(D46-Pad1) -> row3
- D56 pad 1: Net-(D46-Pad1) -> row3
- D57 pad 1: Net-(D46-Pad1) -> row3
- D58 pad 1: Net-(D46-Pad1) -> row3
- D59 pad 1: Net-(D46-Pad1) -> row3
- D6 pad 1: Net-(D1-Pad1) -> row0
- D60 pad 1: Net-(D46-Pad1) -> row3
- D61 pad 1: Net-(D61-Pad1) -> row4
- D62 pad 1: Net-(D61-Pad1) -> row4
- D63 pad 1: Net-(D61-Pad1) -> row4
- D64 pad 1: Net-(D61-Pad1) -> row4
- D65 pad 1: Net-(D61-Pad1) -> row4
- D66 pad 1: Net-(D61-Pad1) -> row4
- D67 pad 1: Net-(D61-Pad1) -> row4
- D68 pad 1: Net-(D61-Pad1) -> row4
- D69 pad 1: Net-(D61-Pad1) -> row4
- D7 pad 1: Net-(D1-Pad1) -> row0
- D8 pad 1: Net-(D1-Pad1) -> row0
- D9 pad 1: Net-(D1-Pad1) -> row0
- K1 pad 1: Net-(K1-Pad1) -> col0
- K10 pad 1: Net-(K10-Pad1) -> col9
- K11 pad 1: Net-(K11-Pad1) -> col10
- K12 pad 1: Net-(K12-Pad1) -> col11
- K13 pad 1: Net-(K13-Pad1) -> col12
- K14 pad 1: Net-(K14-Pad1) -> col13
- K15 pad 1: Net-(K15-Pad1) -> col14
- K16 pad 1: Net-(K16-Pad1) -> col15
- K17 pad 1: Net-(K15-Pad1) -> col14
- K18 pad 1: Net-(K1-Pad1) -> col0
- K19 pad 1: Net-(K19-Pad1) -> col1
- K2 pad 1: Net-(K19-Pad1) -> col1
- K20 pad 1: Net-(K20-Pad1) -> col2
- K21 pad 1: Net-(K21-Pad1) -> col4
- K22 pad 1: Net-(K22-Pad1) -> col5
- K23 pad 1: Net-(K23-Pad1) -> col6
- K24 pad 1: Net-(K24-Pad1) -> col7
- K25 pad 1: Net-(K25-Pad1) -> col8
- K26 pad 1: Net-(K10-Pad1) -> col9
- K27 pad 1: Net-(K11-Pad1) -> col10
- K28 pad 1: Net-(K12-Pad1) -> col11
- K29 pad 1: Net-(K13-Pad1) -> col12
- K3 pad 1: Net-(K20-Pad1) -> col2
- K30 pad 1: Net-(K14-Pad1) -> col13
- K31 pad 1: Net-(K15-Pad1) -> col14
- K32 pad 1: Net-(K16-Pad1) -> col15
- K33 pad 1: Net-(K1-Pad1) -> col0
- K34 pad 1: Net-(K19-Pad1) -> col1
- K35 pad 1: Net-(K20-Pad1) -> col2
- K36 pad 1: Net-(K21-Pad1) -> col4
- K37 pad 1: Net-(K22-Pad1) -> col5
- K38 pad 1: Net-(K23-Pad1) -> col6
- K39 pad 1: Net-(K24-Pad1) -> col7
- K4 pad 1: Net-(K4-Pad1) -> col3
- K40 pad 1: Net-(K25-Pad1) -> col8
- K41 pad 1: Net-(K10-Pad1) -> col9
- K42 pad 1: Net-(K11-Pad1) -> col10
- K43 pad 1: Net-(K12-Pad1) -> col11
- K44 pad 1: Net-(K14-Pad1) -> col13
- K45 pad 1: Net-(K15-Pad1) -> col14
- K46 pad 1: Net-(K16-Pad1) -> col15
- K47 pad 1: Net-(K1-Pad1) -> col0
- K48 pad 1: Net-(K19-Pad1) -> col1
- K49 pad 1: Net-(K20-Pad1) -> col2
- K5 pad 1: Net-(K21-Pad1) -> col4
- K50 pad 1: Net-(K21-Pad1) -> col4
- K51 pad 1: Net-(K22-Pad1) -> col5
- K52 pad 1: Net-(K23-Pad1) -> col6
- K53 pad 1: Net-(K24-Pad1) -> col7
- K54 pad 1: Net-(K25-Pad1) -> col8
- K55 pad 1: Net-(K10-Pad1) -> col9
- K56 pad 1: Net-(K11-Pad1) -> col10
- K57 pad 1: Net-(K12-Pad1) -> col11
- K58 pad 1: Net-(K13-Pad1) -> col12
- K59 pad 1: Net-(K14-Pad1) -> col13
- K6 pad 1: Net-(K22-Pad1) -> col5
- K60 pad 1: Net-(K15-Pad1) -> col14
- K61 pad 1: Net-(K16-Pad1) -> col15
- K62 pad 1: Net-(K15-Pad1) -> col14
- K63 pad 2: Net-(K12-Pad1) -> col11
- K64 pad 1: Net-(K23-Pad1) -> col6
- K65 pad 1: Net-(K24-Pad1) -> col7
- K66 pad 1: Net-(K1-Pad1) -> col0
- K67 pad 1: Net-(K19-Pad1) -> col1
- K68 pad 1: Net-(K21-Pad1) -> col4
- K69 pad 1: Net-(K23-Pad1) -> col6
- K7 pad 1: Net-(K23-Pad1) -> col6
- K70 pad 1: Net-(K24-Pad1) -> col7
- K71 pad 1: Net-(K10-Pad1) -> col9
- K72 pad 1: Net-(K12-Pad1) -> col11
- K73 pad 1: Net-(K14-Pad1) -> col13
- K74 pad 1: Net-(K16-Pad1) -> col15
- K8 pad 1: Net-(K24-Pad1) -> col7
- K9 pad 1: Net-(K25-Pad1) -> col8
- U1 pad 1: Net-(U1-Pad1) -> col8
- U1 pad 10: Net-(U1-Pad10) -> col12
- U1 pad 11: Net-(U1-Pad11) -> col13
- U1 pad 12: Net-(U1-Pad12) -> col14
- U1 pad 18: Net-(U1-Pad18) -> col15
- U1 pad 27: Net-(U1-Pad27) -> row4
- U1 pad 28: Net-(U1-Pad28) -> row3
- U1 pad 29: Net-(U1-Pad29) -> row2
- U1 pad 30: Net-(U1-Pad30) -> row1
- U1 pad 31: Net-(U1-Pad31) -> row0
- U1 pad 32: Net-(U1-Pad32) -> col0
- U1 pad 36: Net-(U1-Pad36) -> col1
- U1 pad 37: Net-(U1-Pad37) -> col2
- U1 pad 38: Net-(U1-Pad38) -> col3
- U1 pad 39: Net-(U1-Pad39) -> col4
- U1 pad 40: Net-(U1-Pad40) -> col5
- U1 pad 41: Net-(U1-Pad41) -> col6
- U1 pad 42: Net-(U1-Pad42) -> col7
- U1 pad 7: Net-(U1-Pad7) -> col9
- U1 pad 8: Net-(U1-Pad8) -> col10
- U1 pad 9: Net-(U1-Pad9) -> col11
Routing:
- net row3: track 0.00 -> 424.0 mm
- net row4: track 0.00 -> 405.8 mm, vias 0 -> 2
- net row2: track 0.00 -> 371.6 mm, vias 0 -> 2
- net row0: track 0.00 -> 368.1 mm, vias 0 -> 4
- net Net-(D46-Pad1): track 365.9 -> 0.00 mm
- net row1: track 0.00 -> 346.1 mm, vias 0 -> 3
- net Net-(D61-Pad1): track 343.2 -> 0.00 mm
- net Net-(D1-Pad1): track 342.8 -> 0.00 mm, vias 2 -> 0
- net Net-(D32-Pad1): track 337.9 -> 0.00 mm, vias 2 -> 0
- net Net-(D17-Pad1): track 337.5 -> 0.00 mm, vias 2 -> 0
- net col15: track 0.00 -> 284.2 mm, vias 0 -> 2
- net col14: track 0.00 -> 242.7 mm
- net col0: track 0.00 -> 238.1 mm
- net col1: track 0.00 -> 214.0 mm, vias 0 -> 2
- net col13: track 0.00 -> 209.3 mm, vias 0 -> 1
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
Commit message: alice
Parts:
- moved K64 0.10 mm to (248.9, 206.7)
Routing:
- net row2: track 371.6 -> 378.8 mm
- added copper zone on B.Cu, net GND
- added copper zone on F.Cu, net GND

Commit message: alice
Parts:
- added J2: AVR-ISP-6, Connectors:2X3, B.Cu at (304.1, 172.9)
Routing:
- net Net-(J2-Pad5): track 33.1 -> 55.9 mm, vias 0 -> 3
- net GND: track 227.3 -> 239.4 mm, vias 7 -> 8
- net VCC: track 145.3 -> 155.4 mm, vias 0 -> 1
- net col12: track 158.8 -> 168.0 mm
- net col11: track 162.6 -> 168.9 mm, vias 0 -> 1
- net col6: track 132.4 -> 137.9 mm
- net col7: track 115.4 -> 119.5 mm
- net Net-(D64-Pad2): track 12.3 -> 14.8 mm
- net row2: track 378.8 -> 381.3 mm
- net Net-(D65-Pad2): track 11.6 -> 14.0 mm
- net Net-(D62-Pad2): track 12.2 -> 14.6 mm
- net col13: track 209.3 -> 211.3 mm
- net col3: track 125.8 -> 127.3 mm
- net row1: track 346.1 -> 345.0 mm
- net row3: track 424.0 -> 423.5 mm
