File: alice/alice/alice.sch (KiCad schematic (older format))
At the start: 159 parts, among them J1 USB_mini_micro_B, K1 KEYSW, K10 KEYSW, K11 KEYSW, K12 KEYSW, K13 KEYSW, K14 KEYSW, K15 KEYSW, K16 KEYSW, K17 KEYSW, K18 KEYSW, K19 KEYSW, K2 KEYSW, K20 KEYSW, K21 KEYSW, K22 KEYSW, K23 KEYSW, K24 KEYSW, K25 KEYSW, K26 KEYSW, K27 KEYSW, K28 KEYSW, K29 KEYSW, K3 KEYSW, K30 KEYSW, K31 KEYSW, K32 KEYSW, K33 KEYSW, K34 KEYSW, K35 KEYSW, K36 KEYSW, K37 KEYSW, K38 KEYSW, K39 KEYSW, K4 KEYSW, K40 KEYSW, K41 KEYSW, K42 KEYSW, K43 KEYSW, K44 KEYSW, K45 KEYSW, K46 KEYSW, K47 KEYSW, K48 KEYSW, K49 KEYSW, K5 KEYSW, K50 KEYSW, K51 KEYSW, K52 KEYSW, K53 KEYSW, K54 KEYSW, K55 KEYSW, K56 KEYSW, K57 KEYSW, K58 KEYSW, K59 KEYSW, K6 KEYSW, K60 KEYSW, K61 KEYSW, K62 KEYSW, K63 KEYSW, K64 KEYSW, K65 KEYSW, K66 KEYSW, K67 KEYSW, K68 KEYSW, K69 KEYSW, K7 KEYSW, K70 KEYSW, K71 KEYSW, K72 KEYSW, K73 KEYSW, K74 KEYSW, K8 KEYSW, K9 KEYSW, SW1 SW_PUSH, U1 ATMEGA32U4, Y1 Crystal_GND24

Commit message: falice
Connections:
- net labels added: col0, col1, col10, col11, col12, col13, col14, col15, col2, col3, col4, col5, col6, col7, col8, col9, row0, row1, row2, row3, row4
Changed lines of the file:
@@
 Connection ~ 11350 8800
 Connection ~ 10600 8800
-Connection ~ 8900 8800
 Connection ~ 8150 8800
 Connection ~ 7400 8800
@@
 Wire Wire Line
 	12250 12800 12250 12950
+Text GLabel 3650 8450 0    50   Input ~ 0
+col0
+Text GLabel 4400 8450 0    50   Input ~ 0
+col1
+Text GLabel 5150 8450 0    50   Input ~ 0
+col2
+Text GLabel 5900 8450 0    50   Input ~ 0
+col3
+Text GLabel 6650 8450 0    50   Input ~ 0
+col4
+Text GLabel 7400 8450 0    50   Input ~ 0
+col5
+Text GLabel 8150 8450 0    50   Input ~ 0
+col6
+Connection ~ 8900 8800
+Text GLabel 8900 8450 0    50   Input ~ 0
+col7
+Text GLabel 10600 8450 0    50   Input ~ 0
+col8
+Text GLabel 11350 8450 0    50   Input ~ 0
+col9
+Text GLabel 12100 8450 0    50   Input ~ 0
+col10
+Text GLabel 12850 8450 0    50   Input ~ 0
+col11
+Text GLabel 13600 8450 0    50   Input ~ 0
+col12
+Text GLabel 14350 8450 0    50   Input ~ 0
+col13
+Text GLabel 15100 8450 0    50   Input ~ 0
+col14
+Text GLabel 15850 8450 0    50   Input ~ 0
+col15
+Text GLabel 2800 9250 0    50   Input ~ 0
+row0
+Text GLabel 2750 10250 0    50   Input ~ 0
+row1
+Text GLabel 2700 11250 0    50   Input ~ 0
+row2
+Text GLabel 2700 12250 0    50   Input ~ 0
+row3
+Text GLabel 2700 13250 0    50   Input ~ 0
+row4
+Text GLabel 5900 4900 2    50   Input ~ 0
+col0
+Text GLabel 5900 4500 2    50   Input ~ 0
+col1
+Text GLabel 5900 4400 2    50   Input ~ 0
+col2
+Text GLabel 5900 4300 2    50   Input ~ 0
+col3
+Text GLabel 5900 4200 2    50   Input ~ 0
+col4
+Text GLabel 5900 4100 2    50   Input ~ 0
+col5
+Text GLabel 5900 4000 2    50   Input ~ 0
+col6
+Text GLabel 5900 3900 2    50   Input ~ 0
+col7
+Text GLabel 3750 3700 0    50   Input ~ 0
+col8
+Text GLabel 3750 4300 0    50   Input ~ 0
+col9
+Text GLabel 3750 4400 0    50   Input ~ 0
+col10
+Text GLabel 3750 4500 0    50   Input ~ 0
+col11
+Text GLabel 3750 4600 0    50   Input ~ 0
+col12
+Text GLabel 3750 4700 0    50   Input ~ 0
+col13
+Text GLabel 3750 4800 0    50   Input ~ 0
+col14
+Text GLabel 3750 5400 0    50   Input ~ 0
+col15
+Text GLabel 5900 5000 2    50   Input ~ 0
+row0
+Text GLabel 5900 5100 2    50   Input ~ 0
+row1
+Text GLabel 5900 5200 2    50   Input ~ 0
+row2
+Text GLabel 5900 5300 2    50   Input ~ 0
+row3
+Text GLabel 5900 5400 2    50   Input ~ 0
+row4
 $EndSCHEMATC

Commit message: alice
Parts:
- added J2: AVR-ISP-6, Connectors:2X3, symbol Connector:AVR-ISP-6
Connections:
- wire segments 281 -> 304
Changed lines of the file:
@@
 Text GLabel 3750 3700 0    50   Input ~ 0
 col8
-Text GLabel 3750 4300 0    50   Input ~ 0
+Text GLabel 3500 4300 0    50   Input ~ 0
 col9
 Text GLabel 3750 4400 0    50   Input ~ 0
 col10
-Text GLabel 3750 4500 0    50   Input ~ 0
+Text GLabel 3100 4350 0    50   Input ~ 0
 col11
-Text GLabel 3750 4600 0    50   Input ~ 0
+Text GLabel 3100 4450 0    50   Input ~ 0
 col12
-Text GLabel 3750 4700 0    50   Input ~ 0
+Text GLabel 3100 4550 0    50   Input ~ 0
 col13
 Text GLabel 3750 4800 0    50   Input ~ 0
@@
 Text GLabel 5900 5400 2    50   Input ~ 0
 row4
+$Comp
+L Connector:AVR-ISP-6 J2
+U 1 1 5BECC2A7
+P 3100 2650
+F 0 "J2" H 2820 2746 50  0000 R CNN
+F 1 "AVR-ISP-6" H 2820 2655 50  0000 R CNN
+F 2 "Connectors:2X3" V 2850 2700 50  0001 C CNN
+F 3 " ~" H 1825 2100 50  0001 C CNN
+	1    3100 2650
+	1    0    0    -1
+$EndComp
+Wire Wire Line
+	3750 4300 3500 4300
+Wire Wire Line
+	3500 2450 3650 2450
+Wire Wire Line
+	3650 2450 3650 4000
+Wire Wire Line
+	3650 4700 3750 4700
+Connection ~ 3650 4000
+Wire Wire Line
+	3650 4000 3650 4700
+Wire Wire Line
+	3750 4600 4200 4600
+Wire Wire Line
+	4200 4600 4200 2550
+Wire Wire Line
+	4200 2550 3500 2550
+Wire Wire Line
+	3750 4500 4100 4500
+Wire Wire Line
+	4100 4500 4100 2650
+Wire Wire Line
+	4100 2650 3500 2650
+Wire Wire Line
+	3750 4500 3200 4500
+Wire Wire Line
+	3200 4500 3200 4350
+Wire Wire Line
+	3200 4350 3100 4350
+Connection ~ 3750 4500
+Wire Wire Line
+	3100 4450 3450 4450
+Wire Wire Line
+	3450 4450 3450 4600
+Wire Wire Line
+	3450 4600 3750 4600
+Connection ~ 3750 4600
+Wire Wire Line
+	3100 4550 3550 4550
+Wire Wire Line
+	3550 4550 3550 4700
+Wire Wire Line
+	3550 4700 3650 4700
+Connection ~ 3650 4700
+Wire Wire Line
+	3500 2750 4000 2750
+Wire Wire Line
+	4000 2750 4000 4900
+Wire Wire Line
+	4000 4900 3750 4900
+Connection ~ 3750 4900
+$Comp
+L power:VCC #PWR0118
+U 1 1 5C09AB1F
+P 3000 2150
+F 0 "#PWR0118" H 3000 2000 50  0001 C CNN
+F 1 "VCC" V 3018 2277 50  0000 L CNN
+F 2 "" H 3000 2150 50  0001 C CNN
+F 3 "" H 3000 2150 50  0001 C CNN
+	1    3000 2150
+	0    1    1    0
+$EndComp
+$Comp
+L power:GND #PWR0119
+U 1 1 5C09AB25
+P 3000 3050
+F 0 "#PWR0119" H 3000 2800 50  0001 C CNN
+F 1 "GND" V 3005 2922 50  0000 R CNN
+F 2 "" H 3000 3050 50  0001 C CNN
+F 3 "" H 3000 3050 50  0001 C CNN
+	1    3000 3050
+	0    -1   -1   0
+$EndComp
 $EndSCHEMATC
